File: STM32F4-MotherBoard_5.0.0/CAN.sch (KiCad schematic (older format))
At the start: 5 parts, among them J1 RJ45, J2 RJ45, U4 MCP2551-I/SN

Commit message: replace project
Connections:
- net +5VP is gone; now on net +12VA: J1.1, J1.2, J2.1, J2.2
- net +12VA: no longer J1.3, J1.4, J2.3, J2.4
- net +5V: now also J1.3, J1.4, J2.3, J2.4
Changed lines of the file:
@@
 LIBS:STM32F4-MotherBoard_3.0.0-cache
 LIBS:STM32F4-MotherBoard_5.0.0-cache
+LIBS:DM3AT-SF-PEJM5
 EELAYER 25 0
 EELAYER END
@@
 	7450 3400 7450 3200
 Wire Wire Line
-	7350 3200 7350 3250
-Wire Wire Line
-	7350 3250 7250 3250
+	7350 3250 7350 3200
+Wire Wire Line
+	7250 3250 7350 3250
 Wire Wire Line
 	7250 3250 7250 3200
@@
 Connection ~ 7300 3250
 Wire Wire Line
-	7150 3200 7150 3250
-Wire Wire Line
-	7150 3250 7050 3250
+	7150 3250 7150 3200
+Wire Wire Line
+	7050 3250 7150 3250
 Wire Wire Line
 	7050 3250 7050 3200
@@
 	7550 3200 7550 3600
 Wire Wire Line
-	9100 3600 5950 3600
+	5950 3600 9100 3600
 $Comp
 L RJ45 J2
@@
 	8900 3250 8900 3200
 Wire Wire Line
-	9000 3200 9000 3400
-Wire Wire Line
-	9100 3200 9100 3600
+	9000 3400 9000 3200
+Wire Wire Line
+	9100 3600 9100 3200
 Wire Wire Line
 	8850 3250 8850 3700
@@
 Connection ~ 8850 3250
 Wire Wire Line
-	9000 3400 5950 3400
+	5950 3400 9000 3400
 Connection ~ 7550 3600
 $Comp
@@
 NoConn ~ 4950 3600
 Wire Wire Line
-	5450 3100 5450 3000
+	5450 3000 5450 3100
 Wire Wire Line
 	5450 3050 6000 3050
@@
 $EndComp
 $Comp
-L +5VP #PWR035
-U 1 1 58A936B6
-P 8150 2800
-F 0 "#PWR035" H 8150 2650 50  0001 C CNN
-F 1 "+5VP" H 8150 2940 50  0000 C CNN
-F 2 "" H 8150 2800 50  0000 C CNN
-F 3 "" H 8150 2800 50  0000 C CNN
-	1    8150 2800
-	1    0    0    -1
-$EndComp
-$Comp
-L +5VP #PWR036
-U 1 1 58A936EF
-P 6600 2800
-F 0 "#PWR036" H 6600 2650 50  0001 C CNN
-F 1 "+5VP" H 6600 2940 50  0000 C CNN
-F 2 "" H 6600 2800 50  0000 C CNN
-F 3 "" H 6600 2800 50  0000 C CNN
-	1    6600 2800
-	1    0    0    -1
-$EndComp
-$Comp
-L +5V #PWR037
+L +5V #PWR035
 U 1 1 58B50836
 P 5450 3000
-F 0 "#PWR037" H 5450 2850 50  0001 C CNN
+F 0 "#PWR035" H 5450 2850 50  0001 C CNN
 F 1 "+5V" H 5450 3140 50  0000 C CNN
 F 2 "" H 5450 3000 50  0000 C CNN
@@
 $EndComp
 $Comp
-L +12VA #PWR038
-U 1 1 58CFCDC9
+L +12VA #PWR036
+U 1 1 58DF64AA
+P 6600 2800
+F 0 "#PWR036" H 6600 2650 50  0001 C CNN
+F 1 "+12VA" H 6600 2940 50  0000 C CNN
+F 2 "" H 6600 2800 50  0000 C CNN
+F 3 "" H 6600 2800 50  0000 C CNN
+	1    6600 2800
+	1    0    0    -1
+$EndComp
+$Comp
+L +12VA #PWR037
+U 1 1 58DF64CB
+P 8150 2800
+F 0 "#PWR037" H 8150 2650 50  0001 C CNN
+F 1 "+12VA" H 8150 2940 50  0000 C CNN
+F 2 "" H 8150 2800 50  0000 C CNN
+F 3 "" H 8150 2800 50  0000 C CNN
+	1    8150 2800
+	1    0    0    -1
+$EndComp
+$Comp
+L +5V #PWR038
+U 1 1 58DF64E2
+P 7950 2800
+F 0 "#PWR038" H 7950 2650 50  0001 C CNN
+F 1 "+5V" H 7950 2940 50  0000 C CNN
+F 2 "" H 7950 2800 50  0000 C CNN
+F 3 "" H 7950 2800 50  0000 C CNN
+	1    7950 2800
+	1    0    0    -1
+$EndComp
+$Comp
+L +5V #PWR039
+U 1 1 58DF6503
 P 6400 2800
-F 0 "#PWR038" H 6400 2650 50  0001 C CNN
-F 1 "+12VA" H 6400 2940 50  0000 C CNN
+F 0 "#PWR039" H 6400 2650 50  0001 C CNN
+F 1 "+5V" H 6400 2940 50  0000 C CNN
 F 2 "" H 6400 2800 50  0000 C CNN
 F 3 "" H 6400 2800 50  0000 C CNN
@@
 	1    0    0    -1
 $EndComp
-$Comp
-L +12VA #PWR039
-U 1 1 58CFCDEA
-P 7950 2800
-F 0 "#PWR039" H 7950 2650 50  0001 C CNN
-F 1 "+12VA" H 7950 2940 50  0000 C CNN
-F 2 "" H 7950 2800 50  0000 C CNN
-F 3 "" H 7950 2800 50  0000 C CNN
-	1    7950 2800
-	1    0    0    -1
-$EndComp
