File: STM32F4-MotherBoard_5.0.0/SW.sch (KiCad schematic (older format))
At the start: 1 part

Commit message: シート作成
Parts:
- removed U?: STM32F407VG, TQFP100, symbol STM32F407VG
Changed lines of the file:
@@
 EELAYER 25 0
 EELAYER END
-$Descr A3 16535 11693
+$Descr A4 11693 8268
 encoding utf-8
-Sheet 1 8
+Sheet 5 8
 Title ""
 Date ""
@@
 Comment4 ""
 $EndDescr
-$Comp
-L STM32F407VG U?
-U 1 1 589AA55C
-P 8063 5478
-F 0 "U?" H 8063 5478 50  0000 C CNN
-F 1 "STM32F407VG" H 8063 5578 50  0000 C CNN
-F 2 "TQFP100" H 8063 5378 50  0000 C CNN
-F 3 "" H 8063 5478 50  0000 C CNN
-	1    8063 5478
-	1    0    0    -1
-$EndComp
-$Sheet
-S 14857 1944 500  150
-U 589AA5CF
-F0 "power" 79
-F1 "power.sch" 79
-$EndSheet
-$Sheet
-S 14851 2334 546  228
-U 589AA5D3
-F0 "CAN" 79
-F1 "CAN.sch" 79
-$EndSheet
-$Sheet
-S 14923 2856 528  188
-U 589AA672
-F0 "RS-232" 79
-F1 "RS-232.sch" 79
-$EndSheet
-$Sheet
-S 15031 3304 500  176
-U 589AA67C
-F0 "SW" 79
-F1 "SW.sch" 79
-$EndSheet
-$Sheet
-S 15072 3762 516  162
-U 589AA689
-F0 "DIO-ADC" 60
-F1 "DIO-ADC.sch" 60
-$EndSheet
-$Sheet
-S 15035 4184 508  150
-U 589AA6A8
-F0 "Display" 79
-F1 "Display.sch" 79
-$EndSheet
-$Sheet
-S 15061 4647 552  165
-U 589AA7A7
-F0 "ST-Link" 79
-F1 "ST-Link.sch" 79
-$EndSheet
 $EndSCHEMATC

Commit message: SW
Parts:
- added C? (x2): 0.1uF, symbol C_Small
- added R? (x5): 10k, symbol R
- added R?: 1k, symbol R
- added SW?: SW_PUSH, symbol SW_PUSH
- added SW?: SW_ROTARY, symbol SW_ROTARY
- added SW?: Reset, symbol SW_PUSH
Connections:
- new net: R?.2, R?.2, SW?.2
- new net +3V3: R?.1, R?.1, R?.1, R?.1, R?.1
- new net GND: C?.2, C?.2, SW?.1, SW?.2, SW?.4 (GND)
- new net NRST: C?.1, SW?.1
- new net PushSW: C?.1, R?.1
- new net RotarySW0: R?.2, SW?.1 (R1)
- new net RotarySW1: R?.2, SW?.2 (R2)
- new net RotarySW2: R?.2, SW?.3 (R4)
- new net RotarySW3: R?.2, SW?.5 (R3)
