File: STM32F4-MotherBoard_5.0.0/SW.sch (KiCad schematic (older format))
At the start: 11 parts

Commit message: add run write
Parts:
- added R?: 10k, symbol R
- added SW?: WRITE/RUN, symbol SW_TOGLE_5P
Connections:
- net +3V3: now also SW?.2
- net GND: now also R?.2, SW?.4
- new net Write: R?.1, SW?.3
Changed lines of the file:
@@
 Text GLabel 2750 4300 0    60   Input ~ 0
 NRST
+Text GLabel 7850 4100 2    60   Input ~ 0
+Write
+$Comp
+L SW_TOGLE_5P SW?
+U 1 1 589F8C6F
+P 7150 4100
+F 0 "SW?" H 7000 4300 60  0000 C CNN
+F 1 "WRITE/RUN" H 6950 3950 60  0000 C CNN
+F 2 "" H 7250 4100 60  0000 C CNN
+F 3 "" H 7250 4100 60  0000 C CNN
+	1    7150 4100
+	-1   0    0    -1
+$EndComp
+$Comp
+L +3.3V #PWR?
+U 1 1 589F8D4E
+P 6500 3750
+F 0 "#PWR?" H 6500 3600 50  0001 C CNN
+F 1 "+3.3V" H 6500 3890 50  0000 C CNN
+F 2 "" H 6500 3750 50  0000 C CNN
+F 3 "" H 6500 3750 50  0000 C CNN
+	1    6500 3750
+	1    0    0    -1
+$EndComp
+Wire Wire Line
+	6500 3750 6500 4000
+Wire Wire Line
+	6500 4000 6650 4000
+Wire Wire Line
+	6650 4200 6500 4200
+Wire Wire Line
+	6500 4200 6500 4500
+Wire Wire Line
+	7750 4100 7750 4150
+$Comp
+L R R?
+U 1 1 589F8E1B
+P 7750 4300
+F 0 "R?" V 7830 4300 50  0000 C CNN
+F 1 "10k" V 7750 4300 50  0000 C CNN
+F 2 "" V 7680 4300 50  0000 C CNN
+F 3 "" H 7750 4300 50  0000 C CNN
+	1    7750 4300
+	1    0    0    -1
+$EndComp
+Wire Wire Line
+	7750 4450 7750 4500
+$Comp
+L GND #PWR?
+U 1 1 589F8EA5
+P 7750 4500
+F 0 "#PWR?" H 7750 4250 50  0001 C CNN
+F 1 "GND" H 7750 4350 50  0000 C CNN
+F 2 "" H 7750 4500 50  0000 C CNN
+F 3 "" H 7750 4500 50  0000 C CNN
+	1    7750 4500
+	1    0    0    -1
+$EndComp
+Wire Wire Line
+	7650 4100 7850 4100
+Connection ~ 7750 4100
+$Comp
+L GND #PWR?
+U 1 1 589F8F49
+P 6500 4500
+F 0 "#PWR?" H 6500 4250 50  0001 C CNN
+F 1 "GND" H 6500 4350 50  0000 C CNN
+F 2 "" H 6500 4500 50  0000 C CNN
+F 3 "" H 6500 4500 50  0000 C CNN
+	1    6500 4500
+	1    0    0    -1
+$EndComp
 $EndSCHEMATC
