File: STM32F4-MotherBoard_5.0.0/SW.sch (KiCad schematic (older format))
At the start: 13 parts

Commit message: 回路図終わり
Parts:
- gave numbers to parts that had none: 13
Changed lines of the file:
@@
 $Descr A4 11693 8268
 encoding utf-8
-Sheet 5 11
+Sheet 5 12
 Title ""
 Date ""
@@
 $EndDescr
 $Comp
-L +3.3V #PWR?
+L +3.3V #PWR041
 U 1 1 589F1FF1
 P 4250 2200
-F 0 "#PWR?" H 4250 2050 50  0001 C CNN
+F 0 "#PWR041" H 4250 2050 50  0001 C CNN
 F 1 "+3.3V" H 4250 2340 50  0000 C CNN
 F 2 "" H 4250 2200 50  0000 C CNN
@@
 $EndComp
 $Comp
-L R R?
+L R R8
 U 1 1 589F2005
 P 4250 2450
-F 0 "R?" V 4330 2450 50  0000 C CNN
+F 0 "R8" V 4330 2450 50  0000 C CNN
 F 1 "10k" V 4250 2450 50  0000 C CNN
 F 2 "" V 4180 2450 50  0000 C CNN
@@
 $EndComp
 $Comp
-L SW_PUSH SW?
+L SW_PUSH SW3
 U 1 1 589F2031
 P 4250 3100
-F 0 "SW?" H 4400 3210 50  0000 C CNN
+F 0 "SW3" H 4400 3210 50  0000 C CNN
 F 1 "SW_PUSH" H 4250 3020 50  0000 C CNN
 F 2 "" H 4250 3100 50  0000 C CNN
@@
 $EndComp
 $Comp
-L R R?
+L R R9
 U 1 1 589F206A
 P 4550 2700
-F 0 "R?" V 4630 2700 50  0000 C CNN
+F 0 "R9" V 4630 2700 50  0000 C CNN
 F 1 "1k" V 4550 2700 50  0000 C CNN
 F 2 "" V 4480 2700 50  0000 C CNN
@@
 Connection ~ 4250 2700
 $Comp
-L C_Small C?
+L C_Small C17
 U 1 1 589F20A4
 P 4900 2950
-F 0 "C?" H 4910 3020 50  0000 L CNN
+F 0 "C17" H 4910 3020 50  0000 L CNN
 F 1 "0.1uF" H 4910 2870 50  0000 L CNN
 F 2 "" H 4900 2950 50  0000 C CNN
@@
 	4900 3050 4900 3550
 $Comp
-L GND #PWR?
+L GND #PWR042
 U 1 1 589F2110
 P 4250 3550
-F 0 "#PWR?" H 4250 3300 50  0001 C CNN
+F 0 "#PWR042" H 4250 3300 50  0001 C CNN
 F 1 "GND" H 4250 3400 50  0000 C CNN
 F 2 "" H 4250 3550 50  0000 C CNN
@@
 $EndComp
 $Comp
-L GND #PWR?
+L GND #PWR043
 U 1 1 589F212E
 P 4900 3550
-F 0 "#PWR?" H 4900 3300 50  0001 C CNN
+F 0 "#PWR043" H 4900 3300 50  0001 C CNN
 F 1 "GND" H 4900 3400 50  0000 C CNN
 F 2 "" H 4900 3550 50  0000 C CNN
@@
 PushSW
 $Comp
-L SW_ROTARY SW?
+L SW_ROTARY SW4
 U 1 1 589F232D
 P 6800 2400
-F 0 "SW?" H 6800 2400 60  0000 C CNN
+F 0 "SW4" H 6800 2400 60  0000 C CNN
 F 1 "SW_ROTARY" H 6800 2200 60  0000 C CNN
 F 2 "" H 6800 2400 60  0000 C CNN
@@
 $EndComp
 $Comp
-L +3.3V #PWR?
+L +3.3V #PWR044
 U 1 1 589F2362
 P 7550 1650
-F 0 "#PWR?" H 7550 1500 50  0001 C CNN
+F 0 "#PWR044" H 7550 1500 50  0001 C CNN
 F 1 "+3.3V" H 7550 1790 50  0000 C CNN
 F 2 "" H 7550 1650 50  0000 C CNN
@@
 $EndComp
 $Comp
-L R R?
+L R R10
 U 1 1 589F2380
 P 7550 1950
-F 0 "R?" V 7630 1950 50  0000 C CNN
+F 0 "R10" V 7630 1950 50  0000 C CNN
 F 1 "10k" V 7550 1950 50  0000 C CNN
 F 2 "" V 7480 1950 50  0000 C CNN
@@
 $EndComp
 $Comp
-L R R?
+L R R11
 U 1 1 589F23BF
 P 7700 1950
-F 0 "R?" V 7780 1950 50  0000 C CNN
+F 0 "R11" V 7780 1950 50  0000 C CNN
 F 1 "10k" V 7700 1950 50  0000 C CNN
 F 2 "" V 7630 1950 50  0000 C CNN
@@
 $EndComp
 $Comp
-L R R?
+L R R13
 U 1 1 589F23EA
 P 7850 1950
-F 0 "R?" V 7930 1950 50  0000 C CNN
+F 0 "R13" V 7930 1950 50  0000 C CNN
 F 1 "10k" V 7850 1950 50  0000 C CNN
 F 2 "" V 7780 1950 50  0000 C CNN
@@
 $EndComp
 $Comp
-L R R?
+L R R14
 U 1 1 589F2414
 P 8000 1950
-F 0 "R?" V 8080 1950 50  0000 C CNN
+F 0 "R14" V 8080 1950 50  0000 C CNN
 F 1 "10k" V 8000 1950 50  0000 C CNN
 F 2 "" V 7930 1950 50  0000 C CNN
@@
 	7650 2500 7650 2750
 $Comp
-L GND #PWR?
+L GND #PWR045
 U 1 1 589F2548
 P 7650 2750
-F 0 "#PWR?" H 7650 2500 50  0001 C CNN
+F 0 "#PWR045" H 7650 2500 50  0001 C CNN
 F 1 "GND" H 7650 2600 50  0000 C CNN
 F 2 "" H 7650 2750 50  0000 C CNN
@@
 RotarySW3
 $Comp
-L SW_PUSH SW?
+L SW_PUSH SW2
 U 1 1 589F289A
 P 3300 4300
-F 0 "SW?" H 3450 4410 50  0000 C CNN
+F 0 "SW2" H 3450 4410 50  0000 C CNN
 F 1 "Reset" H 3300 4220 50  0000 C CNN
 F 2 "" H 3300 4300 50  0000 C CNN
@@
 $EndComp
 $Comp
-L C_Small C?
+L C_Small C16
 U 1 1 589F29F9
 P 2900 4550
-F 0 "C?" H 2910 4620 50  0000 L CNN
+F 0 "C16" H 2910 4620 50  0000 L CNN
 F 1 "0.1uF" H 2910 4470 50  0000 L CNN
 F 2 "" H 2900 4550 50  0000 C CNN
@@
 $EndComp
 $Comp
-L GND #PWR?
+L GND #PWR046
 U 1 1 589F2A59
 P 2900 4750
-F 0 "#PWR?" H 2900 4500 50  0001 C CNN
+F 0 "#PWR046" H 2900 4500 50  0001 C CNN
 F 1 "GND" H 2900 4600 50  0000 C CNN
 F 2 "" H 2900 4750 50  0000 C CNN
@@
 $EndComp
 $Comp
-L GND #PWR?
+L GND #PWR047
 U 1 1 589F2A8C
 P 3700 4750
-F 0 "#PWR?" H 3700 4500 50  0001 C CNN
+F 0 "#PWR047" H 3700 4500 50  0001 C CNN
 F 1 "GND" H 3700 4600 50  0000 C CNN
 F 2 "" H 3700 4750 50  0000 C CNN
@@
 Write
 $Comp
-L SW_TOGLE_5P SW?
+L SW_TOGLE_5P SW5
 U 1 1 589F8C6F
 P 7150 4100
-F 0 "SW?" H 7000 4300 60  0000 C CNN
+F 0 "SW5" H 7000 4300 60  0000 C CNN
 F 1 "WRITE/RUN" H 6950 3950 60  0000 C CNN
 F 2 "" H 7250 4100 60  0000 C CNN
@@
 $EndComp
 $Comp
-L +3.3V #PWR?
+L +3.3V #PWR048
 U 1 1 589F8D4E
 P 6500 3750
-F 0 "#PWR?" H 6500 3600 50  0001 C CNN
+F 0 "#PWR048" H 6500 3600 50  0001 C CNN
 F 1 "+3.3V" H 6500 3890 50  0000 C CNN
 F 2 "" H 6500 3750 50  0000 C CNN
@@
 	7750 4100 7750 4150
 $Comp
-L R R?
+L R R12
 U 1 1 589F8E1B
 P 7750 4300
-F 0 "R?" V 7830 4300 50  0000 C CNN
+F 0 "R12" V 7830 4300 50  0000 C CNN
 F 1 "10k" V 7750 4300 50  0000 C CNN
 F 2 "" V 7680 4300 50  0000 C CNN
@@
 	7750 4450 7750 4500
 $Comp
-L GND #PWR?
+L GND #PWR049
 U 1 1 589F8EA5
 P 7750 4500
-F 0 "#PWR?" H 7750 4250 50  0001 C CNN
+F 0 "#PWR049" H 7750 4250 50  0001 C CNN
 F 1 "GND" H 7750 4350 50  0000 C CNN
 F 2 "" H 7750 4500 50  0000 C CNN
@@
 Connection ~ 7750 4100
 $Comp
-L GND #PWR?
+L GND #PWR050
 U 1 1 589F8F49
 P 6500 4500
-F 0 "#PWR?" H 6500 4250 50  0001 C CNN
+F 0 "#PWR050" H 6500 4250 50  0001 C CNN
 F 1 "GND" H 6500 4350 50  0000 C CNN
 F 2 "" H 6500 4500 50  0000 C CNN

Commit message: 部品名変更
Parts:
- C16, C17: footprint (none) -> robocon_pcb:SM0805_EXP0.5mm
- R10, R11, R12, R13, R14, R8, R9: footprint (none) -> robocon_pcb:SM0603_EXP0.5mm
- SW2, SW3: footprint (none) -> robocon_pcb:SW_PUSH
- SW4: footprint (none) -> mylib:RotarySW
- SW5: footprint (none) -> mylib:SW_TOGGLE_5P
Changed lines of the file:
@@
 EESchema Schematic File Version 2
+LIBS:STM32F4-MotherBoard_5.0.0-rescue
 LIBS:power
 LIBS:device
@@
 $EndDescr
 $Comp
-L +3.3V #PWR041
+L +3.3V #PWR043
 U 1 1 589F1FF1
 P 4250 2200
-F 0 "#PWR041" H 4250 2050 50  0001 C CNN
+F 0 "#PWR043" H 4250 2050 50  0001 C CNN
 F 1 "+3.3V" H 4250 2340 50  0000 C CNN
 F 2 "" H 4250 2200 50  0000 C CNN
@@
 F 0 "R8" V 4330 2450 50  0000 C CNN
 F 1 "10k" V 4250 2450 50  0000 C CNN
-F 2 "" V 4180 2450 50  0000 C CNN
+F 2 "robocon_pcb:SM0603_EXP0.5mm" V 4180 2450 50  0001 C CNN
 F 3 "" H 4250 2450 50  0000 C CNN
 	1    4250 2450
@@
 F 0 "SW3" H 4400 3210 50  0000 C CNN
 F 1 "SW_PUSH" H 4250 3020 50  0000 C CNN
-F 2 "" H 4250 3100 50  0000 C CNN
+F 2 "robocon_pcb:SW_PUSH" H 4250 3100 50  0001 C CNN
 F 3 "" H 4250 3100 50  0000 C CNN
 	1    4250 3100
@@
 F 0 "R9" V 4630 2700 50  0000 C CNN
 F 1 "1k" V 4550 2700 50  0000 C CNN
-F 2 "" V 4480 2700 50  0000 C CNN
+F 2 "robocon_pcb:SM0603_EXP0.5mm" V 4480 2700 50  0001 C CNN
 F 3 "" H 4550 2700 50  0000 C CNN
 	1    4550 2700
@@
 F 0 "C17" H 4910 3020 50  0000 L CNN
 F 1 "0.1uF" H 4910 2870 50  0000 L CNN
-F 2 "" H 4900 2950 50  0000 C CNN
+F 2 "robocon_pcb:SM0805_EXP0.5mm" H 4900 2950 50  0001 C CNN
 F 3 "" H 4900 2950 50  0000 C CNN
 	1    4900 2950
@@
 	4900 3050 4900 3550
 $Comp
-L GND #PWR042
+L GND #PWR044
 U 1 1 589F2110
 P 4250 3550
-F 0 "#PWR042" H 4250 3300 50  0001 C CNN
+F 0 "#PWR044" H 4250 3300 50  0001 C CNN
 F 1 "GND" H 4250 3400 50  0000 C CNN
 F 2 "" H 4250 3550 50  0000 C CNN
@@
 $EndComp
 $Comp
-L GND #PWR043
+L GND #PWR045
 U 1 1 589F212E
 P 4900 3550
-F 0 "#PWR043" H 4900 3300 50  0001 C CNN
+F 0 "#PWR045" H 4900 3300 50  0001 C CNN
 F 1 "GND" H 4900 3400 50  0000 C CNN
 F 2 "" H 4900 3550 50  0000 C CNN
@@
 F 0 "SW4" H 6800 2400 60  0000 C CNN
 F 1 "SW_ROTARY" H 6800 2200 60  0000 C CNN
-F 2 "" H 6800 2400 60  0000 C CNN
+F 2 "mylib:RotarySW" H 6800 2400 60  0001 C CNN
 F 3 "" H 6800 2400 60  0000 C CNN
 	1    6800 2400
@@
 $EndComp
 $Comp
-L +3.3V #PWR044
+L +3.3V #PWR046
 U 1 1 589F2362
 P 7550 1650
-F 0 "#PWR044" H 7550 1500 50  0001 C CNN
+F 0 "#PWR046" H 7550 1500 50  0001 C CNN
 F 1 "+3.3V" H 7550 1790 50  0000 C CNN
 F 2 "" H 7550 1650 50  0000 C CNN
@@
 F 0 "R10" V 7630 1950 50  0000 C CNN
 F 1 "10k" V 7550 1950 50  0000 C CNN
-F 2 "" V 7480 1950 50  0000 C CNN
+F 2 "robocon_pcb:SM0603_EXP0.5mm" V 7480 1950 50  0001 C CNN
 F 3 "" H 7550 1950 50  0000 C CNN
 	1    7550 1950
@@
 F 0 "R11" V 7780 1950 50  0000 C CNN
 F 1 "10k" V 7700 1950 50  0000 C CNN
-F 2 "" V 7630 1950 50  0000 C CNN
+F 2 "robocon_pcb:SM0603_EXP0.5mm" V 7630 1950 50  0001 C CNN
 F 3 "" H 7700 1950 50  0000 C CNN
 	1    7700 1950
@@
 F 0 "R13" V 7930 1950 50  0000 C CNN
 F 1 "10k" V 7850 1950 50  0000 C CNN
-F 2 "" V 7780 1950 50  0000 C CNN
+F 2 "robocon_pcb:SM0603_EXP0.5mm" V 7780 1950 50  0001 C CNN
 F 3 "" H 7850 1950 50  0000 C CNN
 	1    7850 1950
@@
 F 0 "R14" V 8080 1950 50  0000 C CNN
 F 1 "10k" V 8000 1950 50  0000 C CNN
-F 2 "" V 7930 1950 50  0000 C CNN
+F 2 "robocon_pcb:SM0603_EXP0.5mm" V 7930 1950 50  0001 C CNN
 F 3 "" H 8000 1950 50  0000 C CNN
 	1    8000 1950
@@
 	7650 2500 7650 2750
 $Comp
-L GND #PWR045
+L GND #PWR047
 U 1 1 589F2548
 P 7650 2750
-F 0 "#PWR045" H 7650 2500 50  0001 C CNN
+F 0 "#PWR047" H 7650 2500 50  0001 C CNN
 F 1 "GND" H 7650 2600 50  0000 C CNN
 F 2 "" H 7650 2750 50  0000 C CNN
@@
 F 0 "SW2" H 3450 4410 50  0000 C CNN
 F 1 "Reset" H 3300 4220 50  0000 C CNN
-F 2 "" H 3300 4300 50  0000 C CNN
+F 2 "robocon_pcb:SW_PUSH" H 3300 4300 50  0001 C CNN
 F 3 "" H 3300 4300 50  0000 C CNN
 	1    3300 4300
@@
 F 0 "C16" H 2910 4620 50  0000 L CNN
 F 1 "0.1uF" H 2910 4470 50  0000 L CNN
-F 2 "" H 2900 4550 50  0000 C CNN
+F 2 "robocon_pcb:SM0805_EXP0.5mm" H 2900 4550 50  0001 C CNN
 F 3 "" H 2900 4550 50  0000 C CNN
 	1    2900 4550
@@
 $EndComp
 $Comp
-L GND #PWR046
+L GND #PWR048
 U 1 1 589F2A59
 P 2900 4750
-F 0 "#PWR046" H 2900 4500 50  0001 C CNN
+F 0 "#PWR048" H 2900 4500 50  0001 C CNN
 F 1 "GND" H 2900 4600 50  0000 C CNN
 F 2 "" H 2900 4750 50  0000 C CNN
@@
 $EndComp
 $Comp
-L GND #PWR047
+L GND #PWR049
 U 1 1 589F2A8C
 P 3700 4750
-F 0 "#PWR047" H 3700 4500 50  0001 C CNN
+F 0 "#PWR049" H 3700 4500 50  0001 C CNN
 F 1 "GND" H 3700 4600 50  0000 C CNN
 F 2 "" H 3700 4750 50  0000 C CNN
@@
 F 0 "SW5" H 7000 4300 60  0000 C CNN
 F 1 "WRITE/RUN" H 6950 3950 60  0000 C CNN
-F 2 "" H 7250 4100 60  0000 C CNN
+F 2 "mylib:SW_TOGGLE_5P" H 7250 4100 60  0001 C CNN
 F 3 "" H 7250 4100 60  0000 C CNN
 	1    7150 4100
@@
 $EndComp
 $Comp
-L +3.3V #PWR048
+L +3.3V #PWR050
 U 1 1 589F8D4E
 P 6500 3750
-F 0 "#PWR048" H 6500 3600 50  0001 C CNN
+F 0 "#PWR050" H 6500 3600 50  0001 C CNN
 F 1 "+3.3V" H 6500 3890 50  0000 C CNN
 F 2 "" H 6500 3750 50  0000 C CNN
@@
 F 0 "R12" V 7830 4300 50  0000 C CNN
 F 1 "10k" V 7750 4300 50  0000 C CNN
-F 2 "" V 7680 4300 50  0000 C CNN
+F 2 "robocon_pcb:SM0603_EXP0.5mm" V 7680 4300 50  0001 C CNN
 F 3 "" H 7750 4300 50  0000 C CNN
 	1    7750 4300
@@
 	7750 4450 7750 4500
 $Comp
-L GND #PWR049
+L GND #PWR051
 U 1 1 589F8EA5
 P 7750 4500
-F 0 "#PWR049" H 7750 4250 50  0001 C CNN
+F 0 "#PWR051" H 7750 4250 50  0001 C CNN
 F 1 "GND" H 7750 4350 50  0000 C CNN
 F 2 "" H 7750 4500 50  0000 C CNN
@@
 Connection ~ 7750 4100
 $Comp
-L GND #PWR050
+L GND #PWR052
 U 1 1 589F8F49
 P 6500 4500
-F 0 "#PWR050" H 6500 4250 50  0001 C CNN
+F 0 "#PWR052" H 6500 4250 50  0001 C CNN
 F 1 "GND" H 6500 4350 50  0000 C CNN
 F 2 "" H 6500 4500 50  0000 C CNN
