File: STM32F4-MotherBoard_5.0.0/DIO-ADC.sch (KiCad schematic (older format))
At the start: 1 part

Commit message: シート作成
Parts:
- removed U?: STM32F407VG, TQFP100, symbol STM32F407VG
Changed lines of the file:
@@
 EELAYER 25 0
 EELAYER END
-$Descr A3 16535 11693
+$Descr A4 11693 8268
 encoding utf-8
-Sheet 1 8
+Sheet 6 8
 Title ""
 Date ""
@@
 Comment4 ""
 $EndDescr
-$Comp
-L STM32F407VG U?
-U 1 1 589AA55C
-P 8063 5478
-F 0 "U?" H 8063 5478 50  0000 C CNN
-F 1 "STM32F407VG" H 8063 5578 50  0000 C CNN
-F 2 "TQFP100" H 8063 5378 50  0000 C CNN
-F 3 "" H 8063 5478 50  0000 C CNN
-	1    8063 5478
-	1    0    0    -1
-$EndComp
-$Sheet
-S 14857 1944 500  150
-U 589AA5CF
-F0 "power" 79
-F1 "power.sch" 79
-$EndSheet
-$Sheet
-S 14851 2334 546  228
-U 589AA5D3
-F0 "CAN" 79
-F1 "CAN.sch" 79
-$EndSheet
-$Sheet
-S 14923 2856 528  188
-U 589AA672
-F0 "RS-232" 79
-F1 "RS-232.sch" 79
-$EndSheet
-$Sheet
-S 15031 3304 500  176
-U 589AA67C
-F0 "SW" 79
-F1 "SW.sch" 79
-$EndSheet
-$Sheet
-S 15072 3762 516  162
-U 589AA689
-F0 "DIO-ADC" 60
-F1 "DIO-ADC.sch" 60
-$EndSheet
-$Sheet
-S 15035 4184 508  150
-U 589AA6A8
-F0 "Display" 79
-F1 "Display.sch" 79
-$EndSheet
-$Sheet
-S 15061 4647 552  165
-U 589AA7A7
-F0 "ST-Link" 79
-F1 "ST-Link.sch" 79
-$EndSheet
 $EndSCHEMATC

Commit message: DIO-ADC
Parts:
- added P?: DIO0, symbol CONN_02X05
- added P?: DIO1, symbol CONN_02X05
- added P?: ADC, symbol CONN_02X05
- added R? (x8): 4.7k, symbol R
- added R? (x8): 8.4k, symbol R
Connections:
- new net: P?.10 (P10), R?.2
- new net: P?.3 (P3), R?.1
- new net: P?.4 (P4), R?.2
- new net: P?.5 (P5), R?.1
- new net: P?.6 (P6), R?.2
- new net: P?.7 (P7), R?.1
- new net: P?.8 (P8), R?.2
- new net: P?.9 (P9), R?.1
- new net +5V: P?.1 (P1), P?.1 (P1), P?.1 (P1)
- new net ADC0: R?.1, R?.2
- new net ADC1: R?.1, R?.1
- new net ADC2: R?.1, R?.2
- new net ADC3: R?.1, R?.1
- new net ADC4: R?.1, R?.2
- new net ADC5: R?.1, R?.1
- new net ADC6: R?.1, R?.2
- new net ADC7: R?.1, R?.1
- new net DIO0_0: P?.3 (P3), P?.3 (P3)
- new net DIO0_1: P?.4 (P4), P?.4 (P4)
- new net DIO0_2: P?.5 (P5), P?.5 (P5)
- new net DIO0_3: P?.6 (P6), P?.6 (P6)
- new net DIO0_4: P?.7 (P7), P?.7 (P7)
- new net DIO0_5: P?.8 (P8), P?.8 (P8)
- new net DIO0_6: P?.9 (P9), P?.9 (P9)
- new net DIO0_7: P?.10 (P10), P?.10 (P10)
- new net GND: P?.2 (P2), P?.2 (P2), P?.2 (P2), R?.2, R?.2, R?.2, R?.2, R?.2, R?.2, R?.2, R?.2
