File: STM32F4-MotherBoard_5.0.0/DIO-ADC.sch (KiCad schematic (older format))
At the start: 19 parts

Commit message: 回路図終わり
Parts:
- gave numbers to parts that had none: 19
Connections:
- net DIO0_0: no longer P5.3 (P3)
- net DIO0_1: no longer P5.4 (P4)
- net DIO0_2: no longer P5.5 (P5)
- net DIO0_3: no longer P5.6 (P6)
- net DIO0_4: no longer P5.7 (P7)
- net DIO0_5: no longer P5.8 (P8)
- net DIO0_6: no longer P5.9 (P9)
- net DIO0_7: no longer P5.10 (P10)
- new net DIO1_0: P5.3 (P3)
- new net DIO1_1: P5.4 (P4)
- new net DIO1_2: P5.5 (P5)
- new net DIO1_3: P5.6 (P6)
- new net DIO1_4: P5.7 (P7)
- new net DIO1_5: P5.8 (P8)
- new net DIO1_6: P5.9 (P9)
- new net DIO1_7: P5.10 (P10)
Changed lines of the file:
@@
 $Descr A4 11693 8268
 encoding utf-8
-Sheet 6 11
+Sheet 6 12
 Title ""
 Date ""
@@
 $EndDescr
 $Comp
-L CONN_02X05 P?
+L CONN_02X05 P3
 U 1 1 589F2DDA
 P 5050 3200
-F 0 "P?" H 5050 3500 50  0000 C CNN
+F 0 "P3" H 5050 3500 50  0000 C CNN
 F 1 "DIO0" H 5050 2900 50  0000 C CNN
 F 2 "" H 5050 2000 50  0000 C CNN
@@
 	4650 3000 4650 2800
 $Comp
-L +5V #PWR?
+L +5V #PWR051
 U 1 1 589F2E96
 P 4650 2800
-F 0 "#PWR?" H 4650 2650 50  0001 C CNN
+F 0 "#PWR051" H 4650 2650 50  0001 C CNN
 F 1 "+5V" H 4650 2940 50  0000 C CNN
 F 2 "" H 4650 2800 50  0000 C CNN
@@
 	5450 3000 5450 3500
 $Comp
-L GND #PWR?
+L GND #PWR052
 U 1 1 589F2EBA
 P 5450 3500
-F 0 "#PWR?" H 5450 3250 50  0001 C CNN
+F 0 "#PWR052" H 5450 3250 50  0001 C CNN
 F 1 "GND" H 5450 3350 50  0000 C CNN
 F 2 "" H 5450 3500 50  0000 C CNN
@@
 $EndComp
 $Comp
-L CONN_02X05 P?
+L CONN_02X05 P5
 U 1 1 589F2EFF
 P 7050 3200
-F 0 "P?" H 7050 3500 50  0000 C CNN
+F 0 "P5" H 7050 3500 50  0000 C CNN
 F 1 "DIO1" H 7050 2900 50  0000 C CNN
 F 2 "" H 7050 2000 50  0000 C CNN
@@
 $EndComp
 Text GLabel 6500 3100 0    60   BiDi ~ 0
-DIO0_0
+DIO1_0
 Text GLabel 6500 3200 0    60   BiDi ~ 0
-DIO0_2
+DIO1_2
 Text GLabel 6500 3300 0    60   BiDi ~ 0
-DIO0_4
+DIO1_4
 Text GLabel 6500 3400 0    60   BiDi ~ 0
-DIO0_6
+DIO1_6
 Text GLabel 7600 3400 2    60   BiDi ~ 0
-DIO0_7
+DIO1_7
 Text GLabel 7600 3300 2    60   BiDi ~ 0
-DIO0_5
+DIO1_5
 Text GLabel 7600 3200 2    60   BiDi ~ 0
-DIO0_3
+DIO1_3
 Text GLabel 7600 3100 2    60   BiDi ~ 0
-DIO0_1
+DIO1_1
 Wire Wire Line
 	7600 3400 7300 3400
@@
 	6650 3000 6650 2800
 $Comp
-L +5V #PWR?
+L +5V #PWR053
 U 1 1 589F2F17
 P 6650 2800
-F 0 "#PWR?" H 6650 2650 50  0001 C CNN
+F 0 "#PWR053" H 6650 2650 50  0001 C CNN
 F 1 "+5V" H 6650 2940 50  0000 C CNN
 F 2 "" H 6650 2800 50  0000 C CNN
@@
 	7450 3000 7450 3500
 $Comp
-L GND #PWR?
+L GND #PWR054
 U 1 1 589F2F1F
 P 7450 3500
-F 0 "#PWR?" H 7450 3250 50  0001 C CNN
+F 0 "#PWR054" H 7450 3250 50  0001 C CNN
 F 1 "GND" H 7450 3350 50  0000 C CNN
 F 2 "" H 7450 3500 50  0000 C CNN
@@
 $EndComp
 $Comp
-L CONN_02X05 P?
+L CONN_02X05 P4
 U 1 1 589F2F6A
 P 5050 4750
-F 0 "P?" H 5050 5050 50  0000 C CNN
+F 0 "P4" H 5050 5050 50  0000 C CNN
 F 1 "ADC" H 5050 4450 50  0000 C CNN
 F 2 "" H 5050 3550 50  0000 C CNN
@@
 	4650 4550 4650 4350
 $Comp
-L +5V #PWR?
+L +5V #PWR055
 U 1 1 589F2F82
 P 4650 4350
-F 0 "#PWR?" H 4650 4200 50  0001 C CNN
+F 0 "#PWR055" H 4650 4200 50  0001 C CNN
 F 1 "+5V" H 4650 4490 50  0000 C CNN
 F 2 "" H 4650 4350 50  0000 C CNN
@@
 	5450 4550 5450 5050
 $Comp
-L GND #PWR?
+L GND #PWR056
 U 1 1 589F2F8A
 P 5450 5050
-F 0 "#PWR?" H 5450 4800 50  0001 C CNN
+F 0 "#PWR056" H 5450 4800 50  0001 C CNN
 F 1 "GND" H 5450 4900 50  0000 C CNN
 F 2 "" H 5450 5050 50  0000 C CNN
@@
 	4600 4650 4800 4650
 $Comp
-L R R?
+L R R19
 U 1 1 589F3102
 P 4450 4650
-F 0 "R?" V 4530 4650 50  0000 C CNN
+F 0 "R19" V 4530 4650 50  0000 C CNN
 F 1 "4.7k" V 4450 4650 50  0000 C CNN
 F 2 "" V 4380 4650 50  0000 C CNN
@@
 $EndComp
 $Comp
-L R R?
+L R R20
 U 1 1 589F312B
 P 4450 4750
-F 0 "R?" V 4530 4750 50  0000 C CNN
+F 0 "R20" V 4530 4750 50  0000 C CNN
 F 1 "4.7k" V 4450 4750 50  0000 C CNN
 F 2 "" V 4380 4750 50  0000 C CNN
@@
 $EndComp
 $Comp
-L R R?
+L R R21
 U 1 1 589F314A
 P 4450 4850
-F 0 "R?" V 4530 4850 50  0000 C CNN
+F 0 "R21" V 4530 4850 50  0000 C CNN
 F 1 "4.7k" V 4450 4850 50  0000 C CNN
 F 2 "" V 4380 4850 50  0000 C CNN
@@
 $EndComp
 $Comp
-L R R?
+L R R22
 U 1 1 589F316C
 P 4450 4950
-F 0 "R?" V 4530 4950 50  0000 C CNN
+F 0 "R22" V 4530 4950 50  0000 C CNN
 F 1 "4.7k" V 4450 4950 50  0000 C CNN
 F 2 "" V 4380 4950 50  0000 C CNN
@@
 $EndComp
 $Comp
-L R R?
+L R R26
 U 1 1 589F3191
 P 5650 4950
-F 0 "R?" V 5730 4950 50  0000 C CNN
+F 0 "R26" V 5730 4950 50  0000 C CNN
 F 1 "4.7k" V 5650 4950 50  0000 C CNN
 F 2 "" V 5580 4950 50  0000 C CNN
@@
 $EndComp
 $Comp
-L R R?
+L R R25
 U 1 1 589F31E5
 P 5650 4850
-F 0 "R?" V 5730 4850 50  0000 C CNN
+F 0 "R25" V 5730 4850 50  0000 C CNN
 F 1 "4.7k" V 5650 4850 50  0000 C CNN
 F 2 "" V 5580 4850 50  0000 C CNN
@@
 $EndComp
 $Comp
-L R R?
+L R R24
 U 1 1 589F3210
 P 5650 4750
-F 0 "R?" V 5730 4750 50  0000 C CNN
+F 0 "R24" V 5730 4750 50  0000 C CNN
 F 1 "4.7k" V 5650 4750 50  0000 C CNN
 F 2 "" V 5580 4750 50  0000 C CNN
@@
 $EndComp
 $Comp
-L R R?
+L R R23
 U 1 1 589F323E
 P 5650 4650
-F 0 "R?" V 5730 4650 50  0000 C CNN
+F 0 "R23" V 5730 4650 50  0000 C CNN
 F 1 "4.7k" V 5650 4650 50  0000 C CNN
 F 2 "" V 5580 4650 50  0000 C CNN
@@
 	3800 4650 4300 4650
 $Comp
-L R R?
+L R R15
 U 1 1 589F38D9
 P 3900 5250
-F 0 "R?" V 3980 5250 50  0000 C CNN
+F 0 "R15" V 3980 5250 50  0000 C CNN
 F 1 "8.4k" V 3900 5250 50  0000 C CNN
 F 2 "" V 3830 5250 50  0000 C CNN
@@
 $EndComp
 $Comp
-L R R?
+L R R16
 U 1 1 589F391A
 P 4000 5250
-F 0 "R?" V 4080 5250 50  0000 C CNN
+F 0 "R16" V 4080 5250 50  0000 C CNN
 F 1 "8.4k" V 4000 5250 50  0000 C CNN
 F 2 "" V 3930 5250 50  0000 C CNN
@@
 $EndComp
 $Comp
-L R R?
+L R R17
 U 1 1 589F3951
 P 4100 5250
-F 0 "R?" V 4180 5250 50  0000 C CNN
+F 0 "R17" V 4180 5250 50  0000 C CNN
 F 1 "8.4k" V 4100 5250 50  0000 C CNN
 F 2 "" V 4030 5250 50  0000 C CNN
@@
 $EndComp
 $Comp
-L R R?
+L R R18
 U 1 1 589F398B
 P 4200 5250
-F 0 "R?" V 4280 5250 50  0000 C CNN
+F 0 "R18" V 4280 5250 50  0000 C CNN
 F 1 "8.4k" V 4200 5250 50  0000 C CNN
 F 2 "" V 4130 5250 50  0000 C CNN
@@
 $EndComp
 $Comp
-L R R?
+L R R27
 U 1 1 589F3AE8
 P 5900 5250
-F 0 "R?" V 5980 5250 50  0000 C CNN
+F 0 "R27" V 5980 5250 50  0000 C CNN
 F 1 "8.4k" V 5900 5250 50  0000 C CNN
 F 2 "" V 5830 5250 50  0000 C CNN
@@
 $EndComp
 $Comp
-L R R?
+L R R28
 U 1 1 589F3AEE
 P 6000 5250
-F 0 "R?" V 6080 5250 50  0000 C CNN
+F 0 "R28" V 6080 5250 50  0000 C CNN
 F 1 "8.4k" V 6000 5250 50  0000 C CNN
 F 2 "" V 5930 5250 50  0000 C CNN
@@
 $EndComp
 $Comp
-L R R?
+L R R29
 U 1 1 589F3AF4
 P 6100 5250
-F 0 "R?" V 6180 5250 50  0000 C CNN
+F 0 "R29" V 6180 5250 50  0000 C CNN
 F 1 "8.4k" V 6100 5250 50  0000 C CNN
 F 2 "" V 6030 5250 50  0000 C CNN
@@
 $EndComp
 $Comp
-L R R?
+L R R30
 U 1 1 589F3AFA
 P 6200 5250
-F 0 "R?" V 6280 5250 50  0000 C CNN
+F 0 "R30" V 6280 5250 50  0000 C CNN
 F 1 "8.4k" V 6200 5250 50  0000 C CNN
 F 2 "" V 6130 5250 50  0000 C CNN
@@
 Connection ~ 4200 5450
 $Comp
-L GND #PWR?
+L GND #PWR057
 U 1 1 589F3DEA
 P 4200 5500
-F 0 "#PWR?" H 4200 5250 50  0001 C CNN
+F 0 "#PWR057" H 4200 5250 50  0001 C CNN
 F 1 "GND" H 4200 5350 50  0000 C CNN
 F 2 "" H 4200 5500 50  0000 C CNN
@@
 $EndComp
 $Comp
-L GND #PWR?
+L GND #PWR058
 U 1 1 589F3E35
 P 5900 5500
-F 0 "#PWR?" H 5900 5250 50  0001 C CNN
+F 0 "#PWR058" H 5900 5250 50  0001 C CNN
 F 1 "GND" H 5900 5350 50  0000 C CNN
 F 2 "" H 5900 5500 50  0000 C CNN

Commit message: 部品名変更
Parts:
- P3, P4, P5: footprint (none) -> robocon_pcb:RA-H101TD
- R15, R16, R17, R18, R19, R20, R21, R22, R23, R24, R25, R26, R27, R28, R29, R30: footprint (none) -> robocon_pcb:SM0603_EXP0.5mm
Changed lines of the file:
@@
 EESchema Schematic File Version 2
+LIBS:STM32F4-MotherBoard_5.0.0-rescue
 LIBS:power
 LIBS:device
@@
 F 0 "P3" H 5050 3500 50  0000 C CNN
 F 1 "DIO0" H 5050 2900 50  0000 C CNN
-F 2 "" H 5050 2000 50  0000 C CNN
+F 2 "robocon_pcb:RA-H101TD" H 5050 2000 50  0001 C CNN
 F 3 "" H 5050 2000 50  0000 C CNN
 	1    5050 3200
@@
 	4650 3000 4650 2800
 $Comp
-L +5V #PWR051
+L +5V #PWR053
 U 1 1 589F2E96
 P 4650 2800
-F 0 "#PWR051" H 4650 2650 50  0001 C CNN
+F 0 "#PWR053" H 4650 2650 50  0001 C CNN
 F 1 "+5V" H 4650 2940 50  0000 C CNN
 F 2 "" H 4650 2800 50  0000 C CNN
@@
 	5450 3000 5450 3500
 $Comp
-L GND #PWR052
+L GND #PWR054
 U 1 1 589F2EBA
 P 5450 3500
-F 0 "#PWR052" H 5450 3250 50  0001 C CNN
+F 0 "#PWR054" H 5450 3250 50  0001 C CNN
 F 1 "GND" H 5450 3350 50  0000 C CNN
 F 2 "" H 5450 3500 50  0000 C CNN
@@
 F 0 "P5" H 7050 3500 50  0000 C CNN
 F 1 "DIO1" H 7050 2900 50  0000 C CNN
-F 2 "" H 7050 2000 50  0000 C CNN
+F 2 "robocon_pcb:RA-H101TD" H 7050 2000 50  0001 C CNN
 F 3 "" H 7050 2000 50  0000 C CNN
 	1    7050 3200
@@
 	6650 3000 6650 2800
 $Comp
-L +5V #PWR053
+L +5V #PWR055
 U 1 1 589F2F17
 P 6650 2800
-F 0 "#PWR053" H 6650 2650 50  0001 C CNN
+F 0 "#PWR055" H 6650 2650 50  0001 C CNN
 F 1 "+5V" H 6650 2940 50  0000 C CNN
 F 2 "" H 6650 2800 50  0000 C CNN
@@
 	7450 3000 7450 3500
 $Comp
-L GND #PWR054
+L GND #PWR056
 U 1 1 589F2F1F
 P 7450 3500
-F 0 "#PWR054" H 7450 3250 50  0001 C CNN
+F 0 "#PWR056" H 7450 3250 50  0001 C CNN
 F 1 "GND" H 7450 3350 50  0000 C CNN
 F 2 "" H 7450 3500 50  0000 C CNN
@@
 F 0 "P4" H 5050 5050 50  0000 C CNN
 F 1 "ADC" H 5050 4450 50  0000 C CNN
-F 2 "" H 5050 3550 50  0000 C CNN
+F 2 "robocon_pcb:RA-H101TD" H 5050 3550 50  0001 C CNN
 F 3 "" H 5050 3550 50  0000 C CNN
 	1    5050 4750
@@
 	4650 4550 4650 4350
 $Comp
-L +5V #PWR055
+L +5V #PWR057
 U 1 1 589F2F82
 P 4650 4350
-F 0 "#PWR055" H 4650 4200 50  0001 C CNN
+F 0 "#PWR057" H 4650 4200 50  0001 C CNN
 F 1 "+5V" H 4650 4490 50  0000 C CNN
 F 2 "" H 4650 4350 50  0000 C CNN
@@
 	5450 4550 5450 5050
 $Comp
-L GND #PWR056
+L GND #PWR058
 U 1 1 589F2F8A
 P 5450 5050
-F 0 "#PWR056" H 5450 4800 50  0001 C CNN
+F 0 "#PWR058" H 5450 4800 50  0001 C CNN
 F 1 "GND" H 5450 4900 50  0000 C CNN
 F 2 "" H 5450 5050 50  0000 C CNN
@@
 F 0 "R19" V 4530 4650 50  0000 C CNN
 F 1 "4.7k" V 4450 4650 50  0000 C CNN
-F 2 "" V 4380 4650 50  0000 C CNN
+F 2 "robocon_pcb:SM0603_EXP0.5mm" V 4380 4650 50  0001 C CNN
 F 3 "" H 4450 4650 50  0000 C CNN
 	1    4450 4650
@@
 F 0 "R20" V 4530 4750 50  0000 C CNN
 F 1 "4.7k" V 4450 4750 50  0000 C CNN
-F 2 "" V 4380 4750 50  0000 C CNN
+F 2 "robocon_pcb:SM0603_EXP0.5mm" V 4380 4750 50  0001 C CNN
 F 3 "" H 4450 4750 50  0000 C CNN
 	1    4450 4750
@@
 F 0 "R21" V 4530 4850 50  0000 C CNN
 F 1 "4.7k" V 4450 4850 50  0000 C CNN
-F 2 "" V 4380 4850 50  0000 C CNN
+F 2 "robocon_pcb:SM0603_EXP0.5mm" V 4380 4850 50  0001 C CNN
 F 3 "" H 4450 4850 50  0000 C CNN
 	1    4450 4850
@@
 F 0 "R22" V 4530 4950 50  0000 C CNN
 F 1 "4.7k" V 4450 4950 50  0000 C CNN
-F 2 "" V 4380 4950 50  0000 C CNN
+F 2 "robocon_pcb:SM0603_EXP0.5mm" V 4380 4950 50  0001 C CNN
 F 3 "" H 4450 4950 50  0000 C CNN
 	1    4450 4950
@@
 F 0 "R26" V 5730 4950 50  0000 C CNN
 F 1 "4.7k" V 5650 4950 50  0000 C CNN
-F 2 "" V 5580 4950 50  0000 C CNN
+F 2 "robocon_pcb:SM0603_EXP0.5mm" V 5580 4950 50  0001 C CNN
 F 3 "" H 5650 4950 50  0000 C CNN
 	1    5650 4950
@@
 F 0 "R25" V 5730 4850 50  0000 C CNN
 F 1 "4.7k" V 5650 4850 50  0000 C CNN
-F 2 "" V 5580 4850 50  0000 C CNN
+F 2 "robocon_pcb:SM0603_EXP0.5mm" V 5580 4850 50  0001 C CNN
 F 3 "" H 5650 4850 50  0000 C CNN
 	1    5650 4850
@@
 F 0 "R24" V 5730 4750 50  0000 C CNN
 F 1 "4.7k" V 5650 4750 50  0000 C CNN
-F 2 "" V 5580 4750 50  0000 C CNN
+F 2 "robocon_pcb:SM0603_EXP0.5mm" V 5580 4750 50  0001 C CNN
 F 3 "" H 5650 4750 50  0000 C CNN
 	1    5650 4750
@@
 F 0 "R23" V 5730 4650 50  0000 C CNN
 F 1 "4.7k" V 5650 4650 50  0000 C CNN
-F 2 "" V 5580 4650 50  0000 C CNN
+F 2 "robocon_pcb:SM0603_EXP0.5mm" V 5580 4650 50  0001 C CNN
 F 3 "" H 5650 4650 50  0000 C CNN
 	1    5650 4650
@@
 F 0 "R15" V 3980 5250 50  0000 C CNN
 F 1 "8.4k" V 3900 5250 50  0000 C CNN
-F 2 "" V 3830 5250 50  0000 C CNN
+F 2 "robocon_pcb:SM0603_EXP0.5mm" V 3830 5250 50  0001 C CNN
 F 3 "" H 3900 5250 50  0000 C CNN
 	1    3900 5250
@@
 F 0 "R16" V 4080 5250 50  0000 C CNN
 F 1 "8.4k" V 4000 5250 50  0000 C CNN
-F 2 "" V 3930 5250 50  0000 C CNN
+F 2 "robocon_pcb:SM0603_EXP0.5mm" V 3930 5250 50  0001 C CNN
 F 3 "" H 4000 5250 50  0000 C CNN
 	1    4000 5250
@@
 F 0 "R17" V 4180 5250 50  0000 C CNN
 F 1 "8.4k" V 4100 5250 50  0000 C CNN
-F 2 "" V 4030 5250 50  0000 C CNN
+F 2 "robocon_pcb:SM0603_EXP0.5mm" V 4030 5250 50  0001 C CNN
 F 3 "" H 4100 5250 50  0000 C CNN
 	1    4100 5250
@@
 F 0 "R18" V 4280 5250 50  0000 C CNN
 F 1 "8.4k" V 4200 5250 50  0000 C CNN
-F 2 "" V 4130 5250 50  0000 C CNN
+F 2 "robocon_pcb:SM0603_EXP0.5mm" V 4130 5250 50  0001 C CNN
 F 3 "" H 4200 5250 50  0000 C CNN
 	1    4200 5250
@@
 F 0 "R27" V 5980 5250 50  0000 C CNN
 F 1 "8.4k" V 5900 5250 50  0000 C CNN
-F 2 "" V 5830 5250 50  0000 C CNN
+F 2 "robocon_pcb:SM0603_EXP0.5mm" V 5830 5250 50  0001 C CNN
 F 3 "" H 5900 5250 50  0000 C CNN
 	1    5900 5250
@@
 F 0 "R28" V 6080 5250 50  0000 C CNN
 F 1 "8.4k" V 6000 5250 50  0000 C CNN
-F 2 "" V 5930 5250 50  0000 C CNN
+F 2 "robocon_pcb:SM0603_EXP0.5mm" V 5930 5250 50  0001 C CNN
 F 3 "" H 6000 5250 50  0000 C CNN
 	1    6000 5250
@@
 F 0 "R29" V 6180 5250 50  0000 C CNN
 F 1 "8.4k" V 6100 5250 50  0000 C CNN
-F 2 "" V 6030 5250 50  0000 C CNN
+F 2 "robocon_pcb:SM0603_EXP0.5mm" V 6030 5250 50  0001 C CNN
 F 3 "" H 6100 5250 50  0000 C CNN
 	1    6100 5250
@@
 F 0 "R30" V 6280 5250 50  0000 C CNN
 F 1 "8.4k" V 6200 5250 50  0000 C CNN
-F 2 "" V 6130 5250 50  0000 C CNN
+F 2 "robocon_pcb:SM0603_EXP0.5mm" V 6130 5250 50  0001 C CNN
 F 3 "" H 6200 5250 50  0000 C CNN
 	1    6200 5250
@@
 Connection ~ 4200 5450
 $Comp
-L GND #PWR057
+L GND #PWR059
 U 1 1 589F3DEA
 P 4200 5500
-F 0 "#PWR057" H 4200 5250 50  0001 C CNN
+F 0 "#PWR059" H 4200 5250 50  0001 C CNN
 F 1 "GND" H 4200 5350 50  0000 C CNN
 F 2 "" H 4200 5500 50  0000 C CNN
@@
 $EndComp
 $Comp
-L GND #PWR058
+L GND #PWR060
 U 1 1 589F3E35
 P 5900 5500
-F 0 "#PWR058" H 5900 5250 50  0001 C CNN
+F 0 "#PWR060" H 5900 5250 50  0001 C CNN
 F 1 "GND" H 5900 5350 50  0000 C CNN
 F 2 "" H 5900 5500 50  0000 C CNN
