File: STM32F4-MotherBoard_5.0.0/Display.sch (KiCad schematic (older format))
At the start: 1 part

Commit message: シート作成
Parts:
- removed U?: STM32F407VG, TQFP100, symbol STM32F407VG
Changed lines of the file:
@@
 EELAYER 25 0
 EELAYER END
-$Descr A3 16535 11693
+$Descr A4 11693 8268
 encoding utf-8
-Sheet 1 8
+Sheet 7 8
 Title ""
 Date ""
@@
 Comment4 ""
 $EndDescr
-$Comp
-L STM32F407VG U?
-U 1 1 589AA55C
-P 8063 5478
-F 0 "U?" H 8063 5478 50  0000 C CNN
-F 1 "STM32F407VG" H 8063 5578 50  0000 C CNN
-F 2 "TQFP100" H 8063 5378 50  0000 C CNN
-F 3 "" H 8063 5478 50  0000 C CNN
-	1    8063 5478
-	1    0    0    -1
-$EndComp
-$Sheet
-S 14857 1944 500  150
-U 589AA5CF
-F0 "power" 79
-F1 "power.sch" 79
-$EndSheet
-$Sheet
-S 14851 2334 546  228
-U 589AA5D3
-F0 "CAN" 79
-F1 "CAN.sch" 79
-$EndSheet
-$Sheet
-S 14923 2856 528  188
-U 589AA672
-F0 "RS-232" 79
-F1 "RS-232.sch" 79
-$EndSheet
-$Sheet
-S 15031 3304 500  176
-U 589AA67C
-F0 "SW" 79
-F1 "SW.sch" 79
-$EndSheet
-$Sheet
-S 15072 3762 516  162
-U 589AA689
-F0 "DIO-ADC" 60
-F1 "DIO-ADC.sch" 60
-$EndSheet
-$Sheet
-S 15035 4184 508  150
-U 589AA6A8
-F0 "Display" 79
-F1 "Display.sch" 79
-$EndSheet
-$Sheet
-S 15061 4647 552  165
-U 589AA7A7
-F0 "ST-Link" 79
-F1 "ST-Link.sch" 79
-$EndSheet
 $EndSCHEMATC

Commit message: Display
Parts:
- added R?: 510, symbol R
- added R?: 1k, symbol RVAR
- added R?: 10k, symbol R
- added U?: AS021350D, symbol AS021350D
Connections:
- new net: R?.1, U?.26 (IM0), U?.27 (IM3)
- new net: R?.1, U?.32 (LED3-), U?.33 (LED2-), U?.34 (LED1-)
- new net: R?.1, U?.35 (LED+)
- new net +3V3: R?.2, U?.3 (VCI), U?.4 (VDD)
- new net CS: U?.5 (NCS)
- new net FSMC_D0: U?.9 (D0)
- new net FSMC_D1: U?.10 (D1)
- new net FSMC_D10: U?.19 (D10)
- new net FSMC_D11: U?.20 (D11)
- new net FSMC_D12: U?.21 (D12)
- new net FSMC_D13: U?.22 (D13)
- new net FSMC_D14: U?.23 (D14)
- new net FSMC_D15: U?.24 (D15)
- new net FSMC_D2: U?.11 (D2)
- new net FSMC_D3: U?.12 (D3)
- new net FSMC_D4: U?.13 (D4)
- new net FSMC_D5: U?.14 (D5)
- new net FSMC_D6: U?.15 (D6)
- new net FSMC_D7: U?.16 (D7)
- new net FSMC_D8: U?.17 (D8)
- new net FSMC_D9: U?.18 (D9)
- new net GND: R?.2, R?.2, U?.1 (GND), U?.2 (GND), U?.25 (NRES), U?.39 (GND)
- new net RD: U?.8 (NRD)
- new net RS: U?.6 (RS)
- new net WR: U?.7 (NWR)
- new net XL: U?.29 (XL)
- new net XR: U?.31 (XR)
- new net YB: U?.28 (YB)
- new net YT: U?.30 (YT)
Changed lines of the file:
@@
 Comment4 ""
 $EndDescr
+$Comp
+L AS021350D U?
+U 1 1 589F41CD
+P 5600 2850
+F 0 "U?" H 5600 3000 60  0000 C CNN
+F 1 "AS021350D" H 5600 2900 60  0000 C CNN
+F 2 "" H 5600 2850 60  0000 C CNN
+F 3 "" H 5600 2850 60  0000 C CNN
+	1    5600 2850
+	1    0    0    -1
+$EndComp
+$Comp
+L +3.3V #PWR?
+U 1 1 589F41F4
+P 4800 2550
+F 0 "#PWR?" H 4800 2400 50  0001 C CNN
+F 1 "+3.3V" H 4800 2690 50  0000 C CNN
+F 2 "" H 4800 2550 50  0000 C CNN
+F 3 "" H 4800 2550 50  0000 C CNN
+	1    4800 2550
+	1    0    0    -1
+$EndComp
+Wire Wire Line
+	4800 2550 4800 3250
+Wire Wire Line
+	4800 3250 4900 3250
+Wire Wire Line
+	4900 3150 4800 3150
+Connection ~ 4800 3150
+Wire Wire Line
+	4900 2950 4850 2950
+Wire Wire Line
+	4850 2950 4850 5100
+Wire Wire Line
+	4850 3050 4900 3050
+Wire Wire Line
+	4850 5100 6450 5100
+Connection ~ 4850 3050
+Wire Wire Line
+	6300 4750 6350 4750
+Wire Wire Line
+	6350 3350 6350 5150
+$Comp
+L R R?
+U 1 1 589F424B
+P 6450 4550
+F 0 "R?" V 6530 4550 50  0000 C CNN
+F 1 "510" V 6450 4550 50  0000 C CNN
+F 2 "" V 6380 4550 50  0000 C CNN
+F 3 "" H 6450 4550 50  0000 C CNN
+	1    6450 4550
+	1    0    0    -1
+$EndComp
+Connection ~ 6350 5100
+$Comp
+L GND #PWR?
+U 1 1 589F4284
+P 6350 5150
+F 0 "#PWR?" H 6350 4900 50  0001 C CNN
+F 1 "GND" H 6350 5000 50  0000 C CNN
+F 2 "" H 6350 5150 50  0000 C CNN
+F 3 "" H 6350 5150 50  0000 C CNN
+	1    6350 5150
+	1    0    0    -1
+$EndComp
+Wire Wire Line
+	6450 5100 6450 4700
+Wire Wire Line
+	6450 4050 6450 4400
+Wire Wire Line
+	6450 4250 6300 4250
+Wire Wire Line
+	6300 4150 6450 4150
+Connection ~ 6450 4250
+Wire Wire Line
+	6300 4050 6450 4050
+Connection ~ 6450 4150
+Wire Wire Line
+	6300 4350 7300 4350
+Wire Wire Line
+	7300 4350 7300 4250
+$Comp
+L RVAR R?
+U 1 1 589F433B
+P 7300 4000
+F 0 "R?" V 7380 3950 50  0000 C CNN
+F 1 "1k" V 7220 4060 50  0000 C CNN
+F 2 "" H 7300 4000 50  0000 C CNN
+F 3 "" H 7300 4000 50  0000 C CNN
+	1    7300 4000
+	-1   0    0    1
+$EndComp
+Wire Wire Line
+	7300 3750 7300 3600
+$Comp
+L +3.3V #PWR?
+U 1 1 589F43A6
+P 7300 3600
+F 0 "#PWR?" H 7300 3450 50  0001 C CNN
+F 1 "+3.3V" H 7300 3740 50  0000 C CNN
+F 2 "" H 7300 3600 50  0000 C CNN
+F 3 "" H 7300 3600 50  0000 C CNN
+	1    7300 3600
+	1    0    0    -1
+$EndComp
+Wire Wire Line
+	4900 3350 4750 3350
+Wire Wire Line
+	4750 3450 4900 3450
+Wire Wire Line
+	4900 3550 4750 3550
+Wire Wire Line
+	4750 3650 4900 3650
+Wire Wire Line
+	4900 3750 4750 3750
+Wire Wire Line
+	4750 3850 4900 3850
+Wire Wire Line
+	4900 3950 4750 3950
+Wire Wire Line
+	4750 4050 4900 4050
+Wire Wire Line
+	4900 4150 4750 4150
+Wire Wire Line
+	4750 4250 4900 4250
+Wire Wire Line
+	4900 4350 4750 4350
+Wire Wire Line
+	4750 4450 4900 4450
+Wire Wire Line
+	4900 4550 4750 4550
+Wire Wire Line
+	4750 4650 4900 4650
+Wire Wire Line
+	4900 4750 4750 4750
+Wire Wire Line
+	4750 4850 4900 4850
+Wire Wire Line
+	6300 2950 6450 2950
+Wire Wire Line
+	6450 3050 6300 3050
+Wire Wire Line
+	6300 3150 6450 3150
+Wire Wire Line
+	6450 3250 6300 3250
+Wire Wire Line
+	6450 3650 6300 3650
+Wire Wire Line
+	6300 3750 6450 3750
+Wire Wire Line
+	6450 3850 6300 3850
+Wire Wire Line
+	6300 3950 6450 3950
+Wire Wire Line
+	6300 3350 6350 3350
+Connection ~ 6350 4750
+Wire Wire Line
+	6300 3450 7050 3450
+Wire Wire Line
+	7050 3450 7050 3600
+Wire Wire Line
+	6300 3550 6400 3550
+Wire Wire Line
+	6400 3550 6400 3450
+Connection ~ 6400 3450
+$Comp
+L R R?
+U 1 1 589F454D
+P 7050 3750
+F 0 "R?" V 7130 3750 50  0000 C CNN
+F 1 "10k" V 7050 3750 50  0000 C CNN
+F 2 "" V 6980 3750 50  0000 C CNN
+F 3 "" H 7050 3750 50  0000 C CNN
+	1    7050 3750
+	1    0    0    -1
+$EndComp
+$Comp
+L GND #PWR?
+U 1 1 589F457E
+P 7050 4050
+F 0 "#PWR?" H 7050 3800 50  0001 C CNN
+F 1 "GND" H 7050 3900 50  0000 C CNN
+F 2 "" H 7050 4050 50  0000 C CNN
+F 3 "" H 7050 4050 50  0000 C CNN
+	1    7050 4050
+	1    0    0    -1
+$EndComp
+Wire Wire Line
+	7050 4050 7050 3900
+Text GLabel 6450 3750 2    60   Input ~ 0
+XL
+Text GLabel 6450 3650 2    60   Input ~ 0
+YB
+Text GLabel 6450 3950 2    60   Input ~ 0
+XR
+Text GLabel 6450 3850 2    60   Input ~ 0
+YT
+Text GLabel 4750 4150 0    60   Input ~ 0
+FSMC_D4
+Text GLabel 4750 4250 0    60   Input ~ 0
+FSMC_D5
+Text GLabel 4750 4350 0    60   Input ~ 0
+FSMC_D6
+Text GLabel 4750 4450 0    60   Input ~ 0
+FSMC_D7
+Text GLabel 4750 4650 0    60   Input ~ 0
+FSMC_D9
+Text GLabel 4750 4550 0    60   Input ~ 0
+FSMC_D8
+Text GLabel 4750 4750 0    60   Input ~ 0
+FSMC_D10
+Text GLabel 4750 4850 0    60   Input ~ 0
+FSMC_D11
+Text GLabel 6450 2950 2    60   Input ~ 0
+FSMC_D12
+Text GLabel 6450 3050 2    60   Input ~ 0
+FSMC_D13
+Text GLabel 6450 3150 2    60   Input ~ 0
+FSMC_D14
+Text GLabel 6450 3250 2    60   Input ~ 0
+FSMC_D15
+Text GLabel 4750 3950 0    60   Input ~ 0
+FSMC_D2
+Text GLabel 4750 4050 0    60   Input ~ 0
+FSMC_D3
+Text GLabel 4750 3750 0    60   Input ~ 0
+FSMC_D0
+Text GLabel 4750 3850 0    60   Input ~ 0
+FSMC_D1
+Text GLabel 4750 3650 0    60   Input ~ 0
+RD
+Text GLabel 4750 3550 0    60   Input ~ 0
+WR
+Text GLabel 4750 3450 0    60   Input ~ 0
+RS
+Text GLabel 4750 3350 0    60   Input ~ 0
+CS
 $EndSCHEMATC
