File: STM32F4-MotherBoard_5.0.0/ST-Link.sch (KiCad schematic (older format))
At the start: 1 part

Commit message: シート作成
Parts:
- removed U?: STM32F407VG, TQFP100, symbol STM32F407VG
Changed lines of the file:
@@
 EELAYER 25 0
 EELAYER END
-$Descr A3 16535 11693
+$Descr A4 11693 8268
 encoding utf-8
-Sheet 1 8
+Sheet 8 8
 Title ""
 Date ""
@@
 Comment4 ""
 $EndDescr
-$Comp
-L STM32F407VG U?
-U 1 1 589AA55C
-P 8063 5478
-F 0 "U?" H 8063 5478 50  0000 C CNN
-F 1 "STM32F407VG" H 8063 5578 50  0000 C CNN
-F 2 "TQFP100" H 8063 5378 50  0000 C CNN
-F 3 "" H 8063 5478 50  0000 C CNN
-	1    8063 5478
-	1    0    0    -1
-$EndComp
-$Sheet
-S 14857 1944 500  150
-U 589AA5CF
-F0 "power" 79
-F1 "power.sch" 79
-$EndSheet
-$Sheet
-S 14851 2334 546  228
-U 589AA5D3
-F0 "CAN" 79
-F1 "CAN.sch" 79
-$EndSheet
-$Sheet
-S 14923 2856 528  188
-U 589AA672
-F0 "RS-232" 79
-F1 "RS-232.sch" 79
-$EndSheet
-$Sheet
-S 15031 3304 500  176
-U 589AA67C
-F0 "SW" 79
-F1 "SW.sch" 79
-$EndSheet
-$Sheet
-S 15072 3762 516  162
-U 589AA689
-F0 "DIO-ADC" 60
-F1 "DIO-ADC.sch" 60
-$EndSheet
-$Sheet
-S 15035 4184 508  150
-U 589AA6A8
-F0 "Display" 79
-F1 "Display.sch" 79
-$EndSheet
-$Sheet
-S 15061 4647 552  165
-U 589AA7A7
-F0 "ST-Link" 79
-F1 "ST-Link.sch" 79
-$EndSheet
 $EndSCHEMATC

Commit message: ST-Link
Parts:
- added P?: SWD, symbol CONN_01X06
- added R? (x4): 22, symbol R
Connections:
- new net: P?.2 (P2), R?.2
- new net: P?.4 (P4), R?.2
- new net: P?.5 (P5), R?.2
- new net: P?.6 (P6), R?.2
- new net GND: P?.3 (P3)
- new net NRST: R?.1
- new net SWCLK: R?.1
- new net SWDIO: R?.1
- new net SWO: R?.1
- no-connect marks 0 -> 1
Changed lines of the file:
@@
 Comment4 ""
 $EndDescr
+$Comp
+L CONN_01X06 P?
+U 1 1 589F4C21
+P 5650 3050
+F 0 "P?" H 5650 3400 50  0000 C CNN
+F 1 "SWD" V 5750 3050 50  0000 C CNN
+F 2 "" H 5650 3050 50  0000 C CNN
+F 3 "" H 5650 3050 50  0000 C CNN
+	1    5650 3050
+	-1   0    0    -1
+$EndComp
+$Comp
+L R R?
+U 1 1 589F4C7C
+P 6100 2900
+F 0 "R?" V 6180 2900 50  0000 C CNN
+F 1 "22" V 6100 2900 50  0000 C CNN
+F 2 "" V 6030 2900 50  0000 C CNN
+F 3 "" H 6100 2900 50  0000 C CNN
+	1    6100 2900
+	0    1    1    0
+$EndComp
+$Comp
+L R R?
+U 1 1 589F4CC4
+P 6100 3100
+F 0 "R?" V 6180 3100 50  0000 C CNN
+F 1 "22" V 6100 3100 50  0000 C CNN
+F 2 "" V 6030 3100 50  0000 C CNN
+F 3 "" H 6100 3100 50  0000 C CNN
+	1    6100 3100
+	0    1    1    0
+$EndComp
+$Comp
+L R R?
+U 1 1 589F4CE0
+P 6100 3200
+F 0 "R?" V 6180 3200 50  0000 C CNN
+F 1 "22" V 6100 3200 50  0000 C CNN
+F 2 "" V 6030 3200 50  0000 C CNN
+F 3 "" H 6100 3200 50  0000 C CNN
+	1    6100 3200
+	0    1    1    0
+$EndComp
+$Comp
+L R R?
+U 1 1 589F4D03
+P 6100 3300
+F 0 "R?" V 6180 3300 50  0000 C CNN
+F 1 "22" V 6100 3300 50  0000 C CNN
+F 2 "" V 6030 3300 50  0000 C CNN
+F 3 "" H 6100 3300 50  0000 C CNN
+	1    6100 3300
+	0    1    1    0
+$EndComp
+Wire Wire Line
+	5950 3300 5850 3300
+Wire Wire Line
+	5850 3200 5950 3200
+Wire Wire Line
+	5950 3100 5850 3100
+Wire Wire Line
+	5950 2900 5850 2900
+Wire Wire Line
+	6250 2900 6350 2900
+Wire Wire Line
+	6250 3100 6350 3100
+Wire Wire Line
+	6350 3200 6250 3200
+Wire Wire Line
+	6250 3300 6350 3300
+Text GLabel 6350 2900 2    60   Input ~ 0
+SWCLK
+NoConn ~ 5850 2800
+Wire Wire Line
+	5850 3000 5900 3000
+Wire Wire Line
+	5900 3000 5900 3400
+$Comp
+L GND #PWR?
+U 1 1 589F4E4F
+P 5900 3400
+F 0 "#PWR?" H 5900 3150 50  0001 C CNN
+F 1 "GND" H 5900 3250 50  0000 C CNN
+F 2 "" H 5900 3400 50  0000 C CNN
+F 3 "" H 5900 3400 50  0000 C CNN
+	1    5900 3400
+	1    0    0    -1
+$EndComp
+Text GLabel 6350 3100 2    60   Input ~ 0
+SWDIO
+Text GLabel 6350 3200 2    60   Input ~ 0
+NRST
+Text GLabel 6350 3300 2    60   Input ~ 0
+SWO
 $EndSCHEMATC
