File: STM32F4-MotherBoard_5.0.0/power.sch (KiCad schematic (older format))
At the start: 1 part

Commit message: シート作成
Parts:
- removed U?: STM32F407VG, TQFP100, symbol STM32F407VG
Changed lines of the file:
@@
 EELAYER 25 0
 EELAYER END
-$Descr A3 16535 11693
+$Descr A4 11693 8268
 encoding utf-8
-Sheet 1 8
+Sheet 2 8
 Title ""
 Date ""
@@
 Comment4 ""
 $EndDescr
-$Comp
-L STM32F407VG U?
-U 1 1 589AA55C
-P 8063 5478
-F 0 "U?" H 8063 5478 50  0000 C CNN
-F 1 "STM32F407VG" H 8063 5578 50  0000 C CNN
-F 2 "TQFP100" H 8063 5378 50  0000 C CNN
-F 3 "" H 8063 5478 50  0000 C CNN
-	1    8063 5478
-	1    0    0    -1
-$EndComp
-$Sheet
-S 14857 1944 500  150
-U 589AA5CF
-F0 "power" 79
-F1 "power.sch" 79
-$EndSheet
-$Sheet
-S 14851 2334 546  228
-U 589AA5D3
-F0 "CAN" 79
-F1 "CAN.sch" 79
-$EndSheet
-$Sheet
-S 14923 2856 528  188
-U 589AA672
-F0 "RS-232" 79
-F1 "RS-232.sch" 79
-$EndSheet
-$Sheet
-S 15031 3304 500  176
-U 589AA67C
-F0 "SW" 79
-F1 "SW.sch" 79
-$EndSheet
-$Sheet
-S 15072 3762 516  162
-U 589AA689
-F0 "DIO-ADC" 60
-F1 "DIO-ADC.sch" 60
-$EndSheet
-$Sheet
-S 15035 4184 508  150
-U 589AA6A8
-F0 "Display" 79
-F1 "Display.sch" 79
-$EndSheet
-$Sheet
-S 15061 4647 552  165
-U 589AA7A7
-F0 "ST-Link" 79
-F1 "ST-Link.sch" 79
-$EndSheet
 $EndSCHEMATC

Commit message: power
Parts:
- added C?: 10uF, symbol C
- added C?: 22uF, symbol C
- added C?: 0.1uF, symbol C_Small
- added C?: 47uF, symbol C_Small
- added C?: 0.1uF, symbol C
- added P?: VCC, symbol CONN_01X01
- added P?: GND, symbol CONN_01X01
- added R?: 1k, symbol R
- added R?: 330, symbol R
- added R?: 100k, symbol R
- added R?: 10k, symbol R
- added SW?: ON/OFF, symbol SW_TOGLE_5P
- added U?: OKL-T6-W12, symbol OKL-T6-W12
- added U?: PQ033EZ1H, SC-63, symbol PQ033EZ1H
Connections:
- new net: R?.1, SW?.3, U?.1 (ON/OFF)
- new net: R?.2, U?.10 (PowerGood)
- new net: R?.1, U?.6 (Trim)
- new net: R?.1, R?.2
- new net: P?.1 (P1), SW?.4
- new net +12V: C?.1, U?.2 (Vin)
- new net +3V3: C?.1, C?.2, C?.2, R?.1, U?.3 (Vout)
- new net +5V: C?.1, C?.1, U?.1 (Vin), U?.2 (ON/OFF), U?.4 (Vout), U?.5 (Sense)
- new net GND: C?.1, C?.2, C?.2, C?.2, P?.1 (P1), R?.2, R?.2, U?.3 (GND), U?.5 (GND), U?.7 (GND)
- no-connect marks 0 -> 1
