File: STM32F4-MotherBoard_5.0.0/power.sch (KiCad schematic (older format))
At the start: 14 parts

Commit message: add LED
Parts:
- added D?: Power, symbol LED
- added R?: 1k, symbol R
Connections:
- net +3V3: now also R?.1
- net GND: now also D?.1 (K)
- new net: D?.2 (A), R?.2
Changed lines of the file:
@@
 Wire Wire Line
 	8650 2100 8650 1950
+$Comp
+L +3.3V #PWR?
+U 1 1 589F7BEB
+P 2850 2500
+F 0 "#PWR?" H 2850 2350 50  0001 C CNN
+F 1 "+3.3V" H 2850 2640 50  0000 C CNN
+F 2 "" H 2850 2500 50  0000 C CNN
+F 3 "" H 2850 2500 50  0000 C CNN
+	1    2850 2500
+	1    0    0    -1
+$EndComp
+$Comp
+L R R?
+U 1 1 589F7CFB
+P 2850 2750
+F 0 "R?" V 2930 2750 50  0000 C CNN
+F 1 "1k" V 2850 2750 50  0000 C CNN
+F 2 "" V 2780 2750 50  0000 C CNN
+F 3 "" H 2850 2750 50  0000 C CNN
+	1    2850 2750
+	1    0    0    -1
+$EndComp
+Wire Wire Line
+	2850 2600 2850 2500
+$Comp
+L LED D?
+U 1 1 589F7D74
+P 2850 3200
+F 0 "D?" H 2850 3300 50  0000 C CNN
+F 1 "Power" H 2850 3100 50  0000 C CNN
+F 2 "" H 2850 3200 50  0000 C CNN
+F 3 "" H 2850 3200 50  0000 C CNN
+	1    2850 3200
+	0    -1   -1   0
+$EndComp
+Wire Wire Line
+	2850 3000 2850 2900
+Wire Wire Line
+	2850 3400 2850 3550
+$Comp
+L GND #PWR?
+U 1 1 589F7E9D
+P 2850 3550
+F 0 "#PWR?" H 2850 3300 50  0001 C CNN
+F 1 "GND" H 2850 3400 50  0000 C CNN
+F 2 "" H 2850 3550 50  0000 C CNN
+F 3 "" H 2850 3550 50  0000 C CNN
+	1    2850 3550
+	1    0    0    -1
+$EndComp
 $EndSCHEMATC

Commit message: 回路図終わり
Parts:
- gave numbers to parts that had none: 16
Connections:
- net +12V: now also P1.1 (P1), SW1.4
Changed lines of the file:
@@
 $Descr A4 11693 8268
 encoding utf-8
-Sheet 2 11
+Sheet 2 12
 Title ""
 Date ""
@@
 $EndDescr
 $Comp
-L OKL-T6-W12 U?
+L OKL-T6-W12 U2
 U 1 1 589F523C
 P 5150 4200
-F 0 "U?" H 5250 3750 60  0000 C CNN
+F 0 "U2" H 5250 3750 60  0000 C CNN
 F 1 "OKL-T6-W12" H 5400 3650 60  0000 C CNN
 F 2 "" H 5150 4200 60  0000 C CNN
@@
 	5050 4650 5050 4900
 $Comp
-L GND #PWR?
+L GND #PWR011
 U 1 1 589F5275
 P 5050 4900
-F 0 "#PWR?" H 5050 4650 50  0001 C CNN
+F 0 "#PWR011" H 5050 4650 50  0001 C CNN
 F 1 "GND" H 5050 4750 50  0000 C CNN
 F 2 "" H 5050 4900 50  0000 C CNN
@@
 	5700 4300 5900 4300
 $Comp
-L R R?
+L R R5
 U 1 1 589F5294
 P 5900 4500
-F 0 "R?" V 5980 4500 50  0000 C CNN
+F 0 "R5" V 5980 4500 50  0000 C CNN
 F 1 "1k" V 5900 4500 50  0000 C CNN
 F 2 "" V 5830 4500 50  0000 C CNN
@@
 	5900 4650 5900 4700
 $Comp
-L R R?
+L R R6
 U 1 1 589F52CA
 P 5900 4850
-F 0 "R?" V 5980 4850 50  0000 C CNN
+F 0 "R6" V 5980 4850 50  0000 C CNN
 F 1 "330" V 5900 4850 50  0000 C CNN
 F 2 "" V 5830 4850 50  0000 C CNN
@@
 	5900 5000 5900 5050
 $Comp
-L GND #PWR?
+L GND #PWR012
 U 1 1 589F531D
 P 5900 5050
-F 0 "#PWR?" H 5900 4800 50  0001 C CNN
+F 0 "#PWR012" H 5900 4800 50  0001 C CNN
 F 1 "GND" H 5900 4900 50  0000 C CNN
 F 2 "" H 5900 5050 50  0000 C CNN
@@
 Connection ~ 5800 3850
 $Comp
-L C C?
+L C C7
 U 1 1 589F5380
 P 6200 4200
-F 0 "C?" H 6225 4300 50  0000 L CNN
+F 0 "C7" H 6225 4300 50  0000 L CNN
 F 1 "10uF" H 6225 4100 50  0000 L CNN
 F 2 "" H 6238 4050 50  0000 C CNN
@@
 	6200 4350 6200 4450
 $Comp
-L GND #PWR?
+L GND #PWR013
 U 1 1 589F53E5
 P 6200 4450
-F 0 "#PWR?" H 6200 4200 50  0001 C CNN
+F 0 "#PWR013" H 6200 4200 50  0001 C CNN
 F 1 "GND" H 6200 4300 50  0000 C CNN
 F 2 "" H 6200 4450 50  0000 C CNN
@@
 $EndComp
 $Comp
-L +5V #PWR?
+L +5V #PWR014
 U 1 1 589F5401
 P 6200 3450
-F 0 "#PWR?" H 6200 3300 50  0001 C CNN
+F 0 "#PWR014" H 6200 3300 50  0001 C CNN
 F 1 "+5V" H 6200 3590 50  0000 C CNN
 F 2 "" H 6200 3450 50  0000 C CNN
@@
 	5900 2850 5900 3450
 $Comp
-L GND #PWR?
+L GND #PWR015
 U 1 1 589F5456
 P 5900 3450
-F 0 "#PWR?" H 5900 3200 50  0001 C CNN
+F 0 "#PWR015" H 5900 3200 50  0001 C CNN
 F 1 "GND" H 5900 3300 50  0000 C CNN
 F 2 "" H 5900 3450 50  0000 C CNN
@@
 $EndComp
 $Comp
-L C C?
+L C C6
 U 1 1 589F5486
 P 5150 3200
-F 0 "C?" H 5175 3300 50  0000 L CNN
+F 0 "C6" H 5175 3300 50  0000 L CNN
 F 1 "22uF" H 5175 3100 50  0000 L CNN
 F 2 "" H 5188 3050 50  0000 C CNN
@@
 Connection ~ 4850 3000
 $Comp
-L +12V #PWR?
+L +12V #PWR016
 U 1 1 589F5530
 P 4850 2850
-F 0 "#PWR?" H 4850 2700 50  0001 C CNN
+F 0 "#PWR016" H 4850 2700 50  0001 C CNN
 F 1 "+12V" H 4850 2990 50  0000 C CNN
 F 2 "" H 4850 2850 50  0000 C CNN
@@
 	4250 4050 4250 3900
 $Comp
-L R R?
+L R R3
 U 1 1 589F5665
 P 4250 3750
-F 0 "R?" V 4330 3750 50  0000 C CNN
+F 0 "R3" V 4330 3750 50  0000 C CNN
 F 1 "100k" V 4250 3750 50  0000 C CNN
 F 2 "" V 4180 3750 50  0000 C CNN
@@
 	4250 3600 4250 3500
 $Comp
-L +3.3V #PWR?
+L +3.3V #PWR017
 U 1 1 589F56DC
 P 4250 3500
-F 0 "#PWR?" H 4250 3350 50  0001 C CNN
+F 0 "#PWR017" H 4250 3350 50  0001 C CNN
 F 1 "+3.3V" H 4250 3640 50  0000 C CNN
 F 2 "" H 4250 3500 50  0000 C CNN
@@
 	4450 2550 5850 2550
 $Comp
-L SW_TOGLE_5P SW?
+L SW_TOGLE_5P SW1
 U 1 1 589F5786
 P 6350 2550
-F 0 "SW?" H 6200 2750 60  0000 C CNN
+F 0 "SW1" H 6200 2750 60  0000 C CNN
 F 1 "ON/OFF" H 6150 2400 60  0000 C CNN
 F 2 "" H 6450 2550 60  0000 C CNN
@@
 NoConn ~ 6850 2450
 $Comp
-L CONN_01X01 P?
+L CONN_01X01 P1
 U 1 1 589F5820
 P 7350 2650
-F 0 "P?" H 7350 2750 50  0000 C CNN
+F 0 "P1" H 7350 2750 50  0000 C CNN
 F 1 "VCC" V 7450 2650 50  0000 C CNN
 F 2 "" H 7350 2650 50  0000 C CNN
@@
 	7150 2650 6850 2650
 $Comp
-L CONN_01X01 P?
+L CONN_01X01 P2
 U 1 1 589F589A
 P 7350 2850
-F 0 "P?" H 7350 2950 50  0000 C CNN
+F 0 "P2" H 7350 2950 50  0000 C CNN
 F 1 "GND" V 7450 2850 50  0000 C CNN
 F 2 "" H 7350 2850 50  0000 C CNN
@@
 Connection ~ 4450 3950
 $Comp
-L R R?
+L R R4
 U 1 1 589F593C
 P 4450 4400
-F 0 "R?" V 4530 4400 50  0000 C CNN
+F 0 "R4" V 4530 4400 50  0000 C CNN
 F 1 "10k" V 4450 4400 50  0000 C CNN
 F 2 "" V 4380 4400 50  0000 C CNN
@@
 	4450 4550 4450 4650
 $Comp
-L GND #PWR?
+L GND #PWR018
 U 1 1 589F5994
 P 4450 4650
-F 0 "#PWR?" H 4450 4400 50  0001 C CNN
+F 0 "#PWR018" H 4450 4400 50  0001 C CNN
 F 1 "GND" H 4450 4500 50  0000 C CNN
 F 2 "" H 4450 4650 50  0000 C CNN
@@
 $EndComp
 $Comp
-L PQ033EZ1H U?
+L PQ033EZ1H U3
 U 1 1 589F5A16
 P 8700 4000
-F 0 "U?" H 9250 4050 60  0000 C CNN
+F 0 "U3" H 9250 4050 60  0000 C CNN
 F 1 "PQ033EZ1H" H 9250 3950 60  0000 C CNN
 F 2 "SC-63" H 9250 3850 30  0000 C CNN
@@
 $EndComp
 $Comp
-L C_Small C?
+L C_Small C8
 U 1 1 589F5AC6
 P 8500 4600
-F 0 "C?" H 8510 4670 50  0000 L CNN
+F 0 "C8" H 8510 4670 50  0000 L CNN
 F 1 "0.1uF" H 8510 4520 50  0000 L CNN
 F 2 "" H 8500 4600 50  0000 C CNN
@@
 $EndComp
 $Comp
-L C_Small C?
+L C_Small C10
 U 1 1 589F5B07
 P 8900 4600
-F 0 "C?" H 8910 4670 50  0000 L CNN
+F 0 "C10" H 8910 4670 50  0000 L CNN
 F 1 "47uF" H 8910 4520 50  0000 L CNN
 F 2 "" H 8900 4600 50  0000 C CNN
@@
 Connection ~ 8500 4400
 $Comp
-L +3.3V #PWR?
+L +3.3V #PWR019
 U 1 1 589F5D4A
 P 8100 4150
-F 0 "#PWR?" H 8100 4000 50  0001 C CNN
+F 0 "#PWR019" H 8100 4000 50  0001 C CNN
 F 1 "+3.3V" H 8100 4290 50  0000 C CNN
 F 2 "" H 8100 4150 50  0000 C CNN
@@
 $EndComp
 $Comp
-L +5V #PWR?
+L +5V #PWR020
 U 1 1 589F5D78
 P 8250 4150
-F 0 "#PWR?" H 8250 4000 50  0001 C CNN
+F 0 "#PWR020" H 8250 4000 50  0001 C CNN
 F 1 "+5V" H 8250 4290 50  0000 C CNN
 F 2 "" H 8250 4150 50  0000 C CNN
@@
 Connection ~ 8900 4400
 $Comp
-L GND #PWR?
+L GND #PWR021
 U 1 1 589F5E4E
 P 9150 4750
-F 0 "#PWR?" H 9150 4500 50  0001 C CNN
+F 0 "#PWR021" H 9150 4500 50  0001 C CNN
 F 1 "GND" H 9150 4600 50  0000 C CNN
 F 2 "" H 9150 4750 50  0000 C CNN
@@
 $EndComp
 $Comp
-L +3.3V #PWR?
+L +3.3V #PWR022
 U 1 1 589F5F32
 P 8650 1950
-F 0 "#PWR?" H 8650 1800 50  0001 C CNN
+F 0 "#PWR022" H 8650 1800 50  0001 C CNN
 F 1 "+3.3V" H 8650 2090 50  0000 C CNN
 F 2 "" H 8650 1950 50  0000 C CNN
@@
 $EndComp
 $Comp
-L C C?
+L C C9
 U 1 1 589F5F60
 P 8650 2250
-F 0 "C?" H 8675 2350 50  0000 L CNN
+F 0 "C9" H 8675 2350 50  0000 L CNN
 F 1 "0.1uF" H 8675 2150 50  0000 L CNN
 F 2 "" H 8688 2100 50  0000 C CNN
@@
 $EndComp
 $Comp
-L GND #PWR?
+L GND #PWR023
 U 1 1 589F5FA5
 P 8650 2600
-F 0 "#PWR?" H 8650 2350 50  0001 C CNN
+F 0 "#PWR023" H 8650 2350 50  0001 C CNN
 F 1 "GND" H 8650 2450 50  0000 C CNN
 F 2 "" H 8650 2600 50  0000 C CNN
@@
 	8650 2100 8650 1950
 $Comp
-L +3.3V #PWR?
+L +3.3V #PWR024
 U 1 1 589F7BEB
 P 2850 2500
-F 0 "#PWR?" H 2850 2350 50  0001 C CNN
+F 0 "#PWR024" H 2850 2350 50  0001 C CNN
 F 1 "+3.3V" H 2850 2640 50  0000 C CNN
 F 2 "" H 2850 2500 50  0000 C CNN
@@
 $EndComp
 $Comp
-L R R?
+L R R2
 U 1 1 589F7CFB
 P 2850 2750
-F 0 "R?" V 2930 2750 50  0000 C CNN
+F 0 "R2" V 2930 2750 50  0000 C CNN
 F 1 "1k" V 2850 2750 50  0000 C CNN
 F 2 "" V 2780 2750 50  0000 C CNN
@@
 	2850 2600 2850 2500
 $Comp
-L LED D?
+L LED D1
 U 1 1 589F7D74
 P 2850 3200
-F 0 "D?" H 2850 3300 50  0000 C CNN
+F 0 "D1" H 2850 3300 50  0000 C CNN
 F 1 "Power" H 2850 3100 50  0000 C CNN
 F 2 "" H 2850 3200 50  0000 C CNN
@@
 	2850 3400 2850 3550
 $Comp
-L GND #PWR?
+L GND #PWR025
 U 1 1 589F7E9D
 P 2850 3550
-F 0 "#PWR?" H 2850 3300 50  0001 C CNN
+F 0 "#PWR025" H 2850 3300 50  0001 C CNN
 F 1 "GND" H 2850 3400 50  0000 C CNN
 F 2 "" H 2850 3550 50  0000 C CNN
@@
 	1    0    0    -1
 $EndComp
+$Comp
+L +12V #PWR026
+U 1 1 58A58ABA
+P 7100 2100
+F 0 "#PWR026" H 7100 1950 50  0001 C CNN
+F 1 "+12V" H 7100 2240 50  0000 C CNN
+F 2 "" H 7100 2100 50  0000 C CNN
+F 3 "" H 7100 2100 50  0000 C CNN
+	1    7100 2100
+	1    0    0    -1
+$EndComp
+Wire Wire Line
+	7100 2100 7100 2650
+Connection ~ 7100 2650
+$Comp
+L +12V #PWR?
+U 1 1 58A5A598
+P 7400 1050
+F 0 "#PWR?" H 7400 900 50  0001 C CNN
+F 1 "+12V" H 7400 1190 50  0000 C CNN
+F 2 "" H 7400 1050 50  0000 C CNN
+F 3 "" H 7400 1050 50  0000 C CNN
+	1    7400 1050
+	1    0    0    -1
+$EndComp
+$Comp
+L +3.3V #PWR?
+U 1 1 58A5A611
+P 7800 1050
+F 0 "#PWR?" H 7800 900 50  0001 C CNN
+F 1 "+3.3V" H 7800 1190 50  0000 C CNN
+F 2 "" H 7800 1050 50  0000 C CNN
+F 3 "" H 7800 1050 50  0000 C CNN
+	1    7800 1050
+	1    0    0    -1
+$EndComp
+Wire Wire Line
+	7400 1050 7400 1200
+Wire Wire Line
+	7400 1200 7150 1200
+Wire Wire Line
+	7150 1200 7150 1050
+Wire Wire Line
+	7800 1050 7800 1200
+Wire Wire Line
+	7800 1200 8100 1200
+Wire Wire Line
+	8100 1200 8100 1050
+$Comp
+L PWR_FLAG #FLG?
+U 1 1 58A5A6DC
+P 8100 1050
+F 0 "#FLG?" H 8100 1145 50  0001 C CNN
+F 1 "PWR_FLAG" H 8100 1230 50  0000 C CNN
+F 2 "" H 8100 1050 50  0000 C CNN
+F 3 "" H 8100 1050 50  0000 C CNN
+	1    8100 1050
+	1    0    0    -1
+$EndComp
+$Comp
+L PWR_FLAG #FLG?
+U 1 1 58A5A71E
+P 7150 1050
+F 0 "#FLG?" H 7150 1145 50  0001 C CNN
+F 1 "PWR_FLAG" H 7150 1230 50  0000 C CNN
+F 2 "" H 7150 1050 50  0000 C CNN
+F 3 "" H 7150 1050 50  0000 C CNN
+	1    7150 1050
+	1    0    0    -1
+$EndComp

Commit message: 部品名変更
Parts:
- C6, C8, C9: footprint (none) -> robocon_pcb:SM0805_EXP0.5mm
- P1, P2: footprint (none) -> SMD_Packages:1Pin
- R2, R3, R4, R5, R6: footprint (none) -> robocon_pcb:SM0603_EXP0.5mm
- SW1: footprint (none) -> mylib:SW_TOGGLE_5P
- U2: footprint (none) -> robocon_pcb:OKL-T6-W12
- U3: footprint SC-63 -> robocon_pcb:PQ033EZ1HZ
Changed lines of the file:
@@
 EESchema Schematic File Version 2
+LIBS:STM32F4-MotherBoard_5.0.0-rescue
 LIBS:power
 LIBS:device
@@
 F 0 "U2" H 5250 3750 60  0000 C CNN
 F 1 "OKL-T6-W12" H 5400 3650 60  0000 C CNN
-F 2 "" H 5150 4200 60  0000 C CNN
+F 2 "robocon_pcb:OKL-T6-W12" H 5150 4200 60  0001 C CNN
 F 3 "" H 5150 4200 60  0000 C CNN
 	1    5150 4200
@@
 F 0 "R5" V 5980 4500 50  0000 C CNN
 F 1 "1k" V 5900 4500 50  0000 C CNN
-F 2 "" V 5830 4500 50  0000 C CNN
+F 2 "robocon_pcb:SM0603_EXP0.5mm" V 5830 4500 50  0001 C CNN
 F 3 "" H 5900 4500 50  0000 C CNN
 	1    5900 4500
@@
 F 0 "R6" V 5980 4850 50  0000 C CNN
 F 1 "330" V 5900 4850 50  0000 C CNN
-F 2 "" V 5830 4850 50  0000 C CNN
+F 2 "robocon_pcb:SM0603_EXP0.5mm" V 5830 4850 50  0001 C CNN
 F 3 "" H 5900 4850 50  0000 C CNN
 	1    5900 4850
@@
 Wire Wire Line
 	5800 4000 5800 3850
-Wire Wire Line
-	5700 3850 6200 3850
 Connection ~ 5800 3850
 $Comp
@@
 F 0 "C7" H 6225 4300 50  0000 L CNN
 F 1 "10uF" H 6225 4100 50  0000 L CNN
-F 2 "" H 6238 4050 50  0000 C CNN
+F 2 "" H 6238 4050 50  0001 C CNN
 F 3 "" H 6200 4200 50  0000 C CNN
 	1    6200 4200
@@
 	1    0    0    -1
 $EndComp
-Connection ~ 6200 3850
 Wire Wire Line
 	5150 3350 5150 3450
@@
 F 0 "C6" H 5175 3300 50  0000 L CNN
 F 1 "22uF" H 5175 3100 50  0000 L CNN
-F 2 "" H 5188 3050 50  0000 C CNN
+F 2 "robocon_pcb:SM0805_EXP0.5mm" H 5188 3050 50  0001 C CNN
 F 3 "" H 5150 3200 50  0000 C CNN
 	1    5150 3200
@@
 F 0 "R3" V 4330 3750 50  0000 C CNN
 F 1 "100k" V 4250 3750 50  0000 C CNN
-F 2 "" V 4180 3750 50  0000 C CNN
+F 2 "robocon_pcb:SM0603_EXP0.5mm" V 4180 3750 50  0001 C CNN
 F 3 "" H 4250 3750 50  0000 C CNN
 	1    4250 3750
@@
 F 0 "SW1" H 6200 2750 60  0000 C CNN
 F 1 "ON/OFF" H 6150 2400 60  0000 C CNN
-F 2 "" H 6450 2550 60  0000 C CNN
+F 2 "mylib:SW_TOGGLE_5P" H 6450 2550 60  0001 C CNN
 F 3 "" H 6450 2550 60  0000 C CNN
 	1    6350 2550
@@
 F 0 "P1" H 7350 2750 50  0000 C CNN
 F 1 "VCC" V 7450 2650 50  0000 C CNN
-F 2 "" H 7350 2650 50  0000 C CNN
+F 2 "SMD_Packages:1Pin" H 7350 2650 50  0001 C CNN
 F 3 "" H 7350 2650 50  0000 C CNN
 	1    7350 2650
@@
 F 0 "P2" H 7350 2950 50  0000 C CNN
 F 1 "GND" V 7450 2850 50  0000 C CNN
-F 2 "" H 7350 2850 50  0000 C CNN
+F 2 "SMD_Packages:1Pin" H 7350 2850 50  0001 C CNN
 F 3 "" H 7350 2850 50  0000 C CNN
 	1    7350 2850
@@
 F 0 "R4" V 4530 4400 50  0000 C CNN
 F 1 "10k" V 4450 4400 50  0000 C CNN
-F 2 "" V 4380 4400 50  0000 C CNN
+F 2 "robocon_pcb:SM0603_EXP0.5mm" V 4380 4400 50  0001 C CNN
 F 3 "" H 4450 4400 50  0000 C CNN
 	1    4450 4400
@@
 F 0 "U3" H 9250 4050 60  0000 C CNN
 F 1 "PQ033EZ1H" H 9250 3950 60  0000 C CNN
-F 2 "SC-63" H 9250 3850 30  0000 C CNN
+F 2 "robocon_pcb:PQ033EZ1HZ" H 9250 3850 30  0000 C CNN
 F 3 "" H 8700 4000 60  0000 C CNN
 	1    8700 4000
@@
 F 0 "C8" H 8510 4670 50  0000 L CNN
 F 1 "0.1uF" H 8510 4520 50  0000 L CNN
-F 2 "" H 8500 4600 50  0000 C CNN
+F 2 "robocon_pcb:SM0805_EXP0.5mm" H 8500 4600 50  0001 C CNN
 F 3 "" H 8500 4600 50  0000 C CNN
 	1    8500 4600
@@
 F 0 "C10" H 8910 4670 50  0000 L CNN
 F 1 "47uF" H 8910 4520 50  0000 L CNN
-F 2 "" H 8900 4600 50  0000 C CNN
+F 2 "" H 8900 4600 50  0001 C CNN
 F 3 "" H 8900 4600 50  0000 C CNN
 	1    8900 4600
@@
 F 0 "C9" H 8675 2350 50  0000 L CNN
 F 1 "0.1uF" H 8675 2150 50  0000 L CNN
-F 2 "" H 8688 2100 50  0000 C CNN
+F 2 "robocon_pcb:SM0805_EXP0.5mm" H 8688 2100 50  0001 C CNN
 F 3 "" H 8650 2250 50  0000 C CNN
 	1    8650 2250
@@
 F 0 "R2" V 2930 2750 50  0000 C CNN
 F 1 "1k" V 2850 2750 50  0000 C CNN
-F 2 "" V 2780 2750 50  0000 C CNN
+F 2 "robocon_pcb:SM0603_EXP0.5mm" V 2780 2750 50  0001 C CNN
 F 3 "" H 2850 2750 50  0000 C CNN
 	1    2850 2750
@@
 F 0 "D1" H 2850 3300 50  0000 C CNN
 F 1 "Power" H 2850 3100 50  0000 C CNN
-F 2 "" H 2850 3200 50  0000 C CNN
+F 2 "" H 2850 3200 50  0001 C CNN
 F 3 "" H 2850 3200 50  0000 C CNN
 	1    2850 3200
@@
 Connection ~ 7100 2650
 $Comp
-L +12V #PWR?
-U 1 1 58A5A598
-P 7400 1050
-F 0 "#PWR?" H 7400 900 50  0001 C CNN
-F 1 "+12V" H 7400 1190 50  0000 C CNN
-F 2 "" H 7400 1050 50  0000 C CNN
-F 3 "" H 7400 1050 50  0000 C CNN
-	1    7400 1050
-	1    0    0    -1
-$EndComp
-$Comp
-L +3.3V #PWR?
-U 1 1 58A5A611
-P 7800 1050
-F 0 "#PWR?" H 7800 900 50  0001 C CNN
-F 1 "+3.3V" H 7800 1190 50  0000 C CNN
-F 2 "" H 7800 1050 50  0000 C CNN
-F 3 "" H 7800 1050 50  0000 C CNN
-	1    7800 1050
-	1    0    0    -1
-$EndComp
-Wire Wire Line
-	7400 1050 7400 1200
-Wire Wire Line
-	7400 1200 7150 1200
-Wire Wire Line
-	7150 1200 7150 1050
-Wire Wire Line
-	7800 1050 7800 1200
-Wire Wire Line
-	7800 1200 8100 1200
-Wire Wire Line
-	8100 1200 8100 1050
-$Comp
-L PWR_FLAG #FLG?
-U 1 1 58A5A6DC
-P 8100 1050
-F 0 "#FLG?" H 8100 1145 50  0001 C CNN
-F 1 "PWR_FLAG" H 8100 1230 50  0000 C CNN
-F 2 "" H 8100 1050 50  0000 C CNN
-F 3 "" H 8100 1050 50  0000 C CNN
-	1    8100 1050
-	1    0    0    -1
-$EndComp
-$Comp
-L PWR_FLAG #FLG?
+L PWR_FLAG #FLG027
 U 1 1 58A5A71E
-P 7150 1050
-F 0 "#FLG?" H 7150 1145 50  0001 C CNN
-F 1 "PWR_FLAG" H 7150 1230 50  0000 C CNN
-F 2 "" H 7150 1050 50  0000 C CNN
-F 3 "" H 7150 1050 50  0000 C CNN
-	1    7150 1050
-	1    0    0    -1
-$EndComp
+P 7450 2150
+F 0 "#FLG027" H 7450 2245 50  0001 C CNN
+F 1 "PWR_FLAG" H 7450 2330 50  0000 C CNN
+F 2 "" H 7450 2150 50  0000 C CNN
+F 3 "" H 7450 2150 50  0000 C CNN
+	1    7450 2150
+	1    0    0    -1
+$EndComp
+Wire Wire Line
+	7450 2150 7450 2300
+Wire Wire Line
+	7450 2300 7100 2300
+Connection ~ 7100 2300
+Wire Wire Line
+	6200 3850 5700 3850
+Connection ~ 6200 3850
+$Comp
+L PWR_FLAG #FLG028
+U 1 1 58A5BB0C
+P 7100 3250
+F 0 "#FLG028" H 7100 3345 50  0001 C CNN
+F 1 "PWR_FLAG" H 7100 3430 50  0000 C CNN
+F 2 "" H 7100 3250 50  0000 C CNN
+F 3 "" H 7100 3250 50  0000 C CNN
+	1    7100 3250
+	1    0    0    -1
+$EndComp
+Wire Wire Line
+	7100 3250 6650 3250
+Wire Wire Line
+	6650 3250 6650 2850
+Connection ~ 6650 2850
 $EndSCHEMATC

Commit message: 関連付けできたの
Parts:
- C10: footprint (none) -> Capacitors_SMD:C_1210_HandSoldering
- C7: footprint (none) -> robocon_pcb:SM0805_EXP0.5mm
- D1: footprint (none) -> LEDs:LED_WS2812B-PLCC4
Changed lines of the file:
@@
 F 0 "C7" H 6225 4300 50  0000 L CNN
 F 1 "10uF" H 6225 4100 50  0000 L CNN
-F 2 "" H 6238 4050 50  0001 C CNN
+F 2 "robocon_pcb:SM0805_EXP0.5mm" H 6238 4050 50  0001 C CNN
 F 3 "" H 6200 4200 50  0000 C CNN
 	1    6200 4200
@@
 F 0 "C10" H 8910 4670 50  0000 L CNN
 F 1 "47uF" H 8910 4520 50  0000 L CNN
-F 2 "" H 8900 4600 50  0001 C CNN
+F 2 "Capacitors_SMD:C_1210_HandSoldering" H 8900 4600 50  0001 C CNN
 F 3 "" H 8900 4600 50  0000 C CNN
 	1    8900 4600
@@
 F 0 "D1" H 2850 3300 50  0000 C CNN
 F 1 "Power" H 2850 3100 50  0000 C CNN
-F 2 "" H 2850 3200 50  0001 C CNN
+F 2 "LEDs:LED_WS2812B-PLCC4" H 2850 3200 50  0001 C CNN
 F 3 "" H 2850 3200 50  0000 C CNN
 	1    2850 3200
