File: STM32F4-MotherBoard_5.0.0/RS-232.sch (KiCad schematic (older format))
At the start: 1 part

Commit message: シート作成
Parts:
- removed U?: STM32F407VG, TQFP100, symbol STM32F407VG
Changed lines of the file:
@@
 EELAYER 25 0
 EELAYER END
-$Descr A3 16535 11693
+$Descr A4 11693 8268
 encoding utf-8
-Sheet 1 8
+Sheet 4 8
 Title ""
 Date ""
@@
 Comment4 ""
 $EndDescr
-$Comp
-L STM32F407VG U?
-U 1 1 589AA55C
-P 8063 5478
-F 0 "U?" H 8063 5478 50  0000 C CNN
-F 1 "STM32F407VG" H 8063 5578 50  0000 C CNN
-F 2 "TQFP100" H 8063 5378 50  0000 C CNN
-F 3 "" H 8063 5478 50  0000 C CNN
-	1    8063 5478
-	1    0    0    -1
-$EndComp
-$Sheet
-S 14857 1944 500  150
-U 589AA5CF
-F0 "power" 79
-F1 "power.sch" 79
-$EndSheet
-$Sheet
-S 14851 2334 546  228
-U 589AA5D3
-F0 "CAN" 79
-F1 "CAN.sch" 79
-$EndSheet
-$Sheet
-S 14923 2856 528  188
-U 589AA672
-F0 "RS-232" 79
-F1 "RS-232.sch" 79
-$EndSheet
-$Sheet
-S 15031 3304 500  176
-U 589AA67C
-F0 "SW" 79
-F1 "SW.sch" 79
-$EndSheet
-$Sheet
-S 15072 3762 516  162
-U 589AA689
-F0 "DIO-ADC" 60
-F1 "DIO-ADC.sch" 60
-$EndSheet
-$Sheet
-S 15035 4184 508  150
-U 589AA6A8
-F0 "Display" 79
-F1 "Display.sch" 79
-$EndSheet
-$Sheet
-S 15061 4647 552  165
-U 589AA7A7
-F0 "ST-Link" 79
-F1 "ST-Link.sch" 79
-$EndSheet
 $EndSCHEMATC

Commit message: RS-232
Parts:
- added C? (x5): 0.1uF, symbol C_Small
- added J? (x2): RJ12, symbol RJ12
- added U?: ADM3202, symbol ADM3202
Connections:
- new net: C?.1, U?.1 (C1+)
- new net: J?.4, U?.13 (R1IN)
- new net: J?.5, U?.14 (T1OUT)
- new net: C?.2, U?.2 (V+)
- new net: C?.2, U?.3 (C1-)
- new net: C?.1, U?.4 (C2+)
- new net: C?.2, U?.5 (C2-)
- new net: C?.1, U?.6 (V-)
- new net: J?.5, U?.7 (T2OUT)
- new net: J?.4, U?.8 (R2IN)
- new net +3V3: C?.1, C?.2, U?.16 (VCC)
- new net +5V: J?.2, J?.2
- new net GND: C?.1, C?.2, J?.3, J?.3, U?.15 (GND)
- new net RS-232(Controller)_RX: U?.12 (R1OUT)
- new net RS-232(Controller)_TX: U?.11 (T1IN)
- new net RS-232(PC)_RX: U?.9 (R2OUT)
- new net RS-232(PC)_TX: U?.10 (T2IN)
- no-connect marks 0 -> 8
