File: STM32F4-MotherBoard_5.0.0/RS-232.sch (KiCad schematic (older format))
At the start: 8 parts

Commit message: 回路図終わり
Parts:
- gave numbers to parts that had none: 8
Changed lines of the file:
@@
 $Descr A4 11693 8268
 encoding utf-8
-Sheet 4 11
+Sheet 4 12
 Title ""
 Date ""
@@
 $EndDescr
 $Comp
-L ADM3202 U?
+L ADM3202 U5
 U 1 1 589F654C
 P 5550 2900
-F 0 "U?" H 5550 3450 60  0000 C CNN
+F 0 "U5" H 5550 3450 60  0000 C CNN
 F 1 "ADM3202" H 5550 2450 60  0000 C CNN
 F 2 "" H 5450 2900 60  0000 C CNN
@@
 $EndComp
 $Comp
-L C_Small C?
+L C_Small C11
 U 1 1 589F6577
 P 4800 2500
-F 0 "C?" H 4810 2570 50  0000 L CNN
+F 0 "C11" H 4810 2570 50  0000 L CNN
 F 1 "0.1uF" H 4810 2420 50  0000 L CNN
 F 2 "" H 4800 2500 50  0000 C CNN
@@
 $EndComp
 $Comp
-L C_Small C?
+L C_Small C12
 U 1 1 589F65AE
 P 4800 2800
-F 0 "C?" H 4810 2870 50  0000 L CNN
+F 0 "C12" H 4810 2870 50  0000 L CNN
 F 1 "0.1uF" H 4810 2720 50  0000 L CNN
 F 2 "" H 4800 2800 50  0000 C CNN
@@
 	4700 2200 5250 2200
 $Comp
-L C_Small C?
+L C_Small C14
 U 1 1 589F661E
 P 5350 2200
-F 0 "C?" H 5360 2270 50  0000 L CNN
+F 0 "C14" H 5360 2270 50  0000 L CNN
 F 1 "0.1uF" H 5360 2120 50  0000 L CNN
 F 2 "" H 5350 2200 50  0000 C CNN
@@
 	6150 2500 6250 2500
 $Comp
-L C_Small C?
+L C_Small C15
 U 1 1 589F6660
 P 6350 2500
-F 0 "C?" H 6360 2570 50  0000 L CNN
+F 0 "C15" H 6360 2570 50  0000 L CNN
 F 1 "0.1uF" H 6360 2420 50  0000 L CNN
 F 2 "" H 6350 2500 50  0000 C CNN
@@
 	6150 2600 6550 2600
 $Comp
-L GND #PWR?
+L GND #PWR034
 U 1 1 589F66C4
 P 6800 2550
-F 0 "#PWR?" H 6800 2300 50  0001 C CNN
+F 0 "#PWR034" H 6800 2300 50  0001 C CNN
 F 1 "GND" H 6800 2400 50  0000 C CNN
 F 2 "" H 6800 2550 50  0000 C CNN
@@
 Connection ~ 6200 2500
 $Comp
-L +3.3V #PWR?
+L +3.3V #PWR035
 U 1 1 589F6792
 P 6200 2100
-F 0 "#PWR?" H 6200 1950 50  0001 C CNN
+F 0 "#PWR035" H 6200 1950 50  0001 C CNN
 F 1 "+3.3V" H 6200 2240 50  0000 C CNN
 F 2 "" H 6200 2100 50  0000 C CNN
@@
 	4950 3000 4900 3000
 $Comp
-L C_Small C?
+L C_Small C13
 U 1 1 589F67EC
 P 4800 3000
-F 0 "C?" H 4810 3070 50  0000 L CNN
+F 0 "C13" H 4810 3070 50  0000 L CNN
 F 1 "0.1uF" H 4810 2920 50  0000 L CNN
 F 2 "" H 4800 3000 50  0000 C CNN
@@
 	4700 3000 4500 3000
 $Comp
-L GND #PWR?
+L GND #PWR036
 U 1 1 589F6831
 P 4500 3000
-F 0 "#PWR?" H 4500 2750 50  0001 C CNN
+F 0 "#PWR036" H 4500 2750 50  0001 C CNN
 F 1 "GND" H 4500 2850 50  0000 C CNN
 F 2 "" H 4500 3000 50  0000 C CNN
@@
 	6300 3000 6150 3000
 $Comp
-L RJ12 J?
+L RJ12 J4
 U 1 1 589F6AEB
 P 3400 2650
-F 0 "J?" H 3600 3150 50  0000 C CNN
+F 0 "J4" H 3600 3150 50  0000 C CNN
 F 1 "RJ12" H 3250 3150 50  0000 C CNN
 F 2 "" H 3400 2650 50  0000 C CNN
@@
 NoConn ~ 3900 2350
 $Comp
-L RJ12 J?
+L RJ12 J3
 U 1 1 589F6B76
 P 2450 2650
-F 0 "J?" H 2650 3150 50  0000 C CNN
+F 0 "J3" H 2650 3150 50  0000 C CNN
 F 1 "RJ12" H 2300 3150 50  0000 C CNN
 F 2 "" H 2450 2650 50  0000 C CNN
@@
 	2450 3100 2450 3150
 $Comp
-L GND #PWR?
+L GND #PWR037
 U 1 1 589F6C63
 P 2450 3150
-F 0 "#PWR?" H 2450 2900 50  0001 C CNN
+F 0 "#PWR037" H 2450 2900 50  0001 C CNN
 F 1 "GND" H 2450 3000 50  0000 C CNN
 F 2 "" H 2450 3150 50  0000 C CNN
@@
 $EndComp
 $Comp
-L GND #PWR?
+L GND #PWR038
 U 1 1 589F6C8D
 P 3400 3150
-F 0 "#PWR?" H 3400 2900 50  0001 C CNN
+F 0 "#PWR038" H 3400 2900 50  0001 C CNN
 F 1 "GND" H 3400 3000 50  0000 C CNN
 F 2 "" H 3400 3150 50  0000 C CNN
@@
 	2950 3200 2950 2900
 $Comp
-L +5V #PWR?
+L +5V #PWR039
 U 1 1 589F6D4F
 P 2950 2900
-F 0 "#PWR?" H 2950 2750 50  0001 C CNN
+F 0 "#PWR039" H 2950 2750 50  0001 C CNN
 F 1 "+5V" H 2950 3040 50  0000 C CNN
 F 2 "" H 2950 2900 50  0000 C CNN
@@
 $EndComp
 $Comp
-L +5V #PWR?
+L +5V #PWR040
 U 1 1 589F6D79
 P 2000 2900
-F 0 "#PWR?" H 2000 2750 50  0001 C CNN
+F 0 "#PWR040" H 2000 2750 50  0001 C CNN
 F 1 "+5V" H 2000 3040 50  0000 C CNN
 F 2 "" H 2000 2900 50  0000 C CNN

Commit message: 部品名変更
Parts:
- C11, C12, C13, C14, C15: footprint (none) -> robocon_pcb:SM0805_EXP0.5mm
- J3, J4: footprint (none) -> robocon_pcb:MODULAR-JACK_6P6C
- U5: footprint (none) -> SMD_Packages:SO-16-N
Changed lines of the file:
@@
 EESchema Schematic File Version 2
+LIBS:STM32F4-MotherBoard_5.0.0-rescue
 LIBS:power
 LIBS:device
@@
 F 0 "U5" H 5550 3450 60  0000 C CNN
 F 1 "ADM3202" H 5550 2450 60  0000 C CNN
-F 2 "" H 5450 2900 60  0000 C CNN
+F 2 "SMD_Packages:SO-16-N" H 5450 2900 60  0001 C CNN
 F 3 "" H 5450 2900 60  0000 C CNN
 	1    5550 2900
@@
 F 0 "C11" H 4810 2570 50  0000 L CNN
 F 1 "0.1uF" H 4810 2420 50  0000 L CNN
-F 2 "" H 4800 2500 50  0000 C CNN
+F 2 "robocon_pcb:SM0805_EXP0.5mm" H 4800 2500 50  0001 C CNN
 F 3 "" H 4800 2500 50  0000 C CNN
 	1    4800 2500
@@
 F 0 "C12" H 4810 2870 50  0000 L CNN
 F 1 "0.1uF" H 4810 2720 50  0000 L CNN
-F 2 "" H 4800 2800 50  0000 C CNN
+F 2 "robocon_pcb:SM0805_EXP0.5mm" H 4800 2800 50  0001 C CNN
 F 3 "" H 4800 2800 50  0000 C CNN
 	1    4800 2800
@@
 F 0 "C14" H 5360 2270 50  0000 L CNN
 F 1 "0.1uF" H 5360 2120 50  0000 L CNN
-F 2 "" H 5350 2200 50  0000 C CNN
+F 2 "robocon_pcb:SM0805_EXP0.5mm" H 5350 2200 50  0001 C CNN
 F 3 "" H 5350 2200 50  0000 C CNN
 	1    5350 2200
@@
 F 0 "C15" H 6360 2570 50  0000 L CNN
 F 1 "0.1uF" H 6360 2420 50  0000 L CNN
-F 2 "" H 6350 2500 50  0000 C CNN
+F 2 "robocon_pcb:SM0805_EXP0.5mm" H 6350 2500 50  0001 C CNN
 F 3 "" H 6350 2500 50  0000 C CNN
 	1    6350 2500
@@
 	6150 2600 6550 2600
 $Comp
-L GND #PWR034
+L GND #PWR036
 U 1 1 589F66C4
 P 6800 2550
-F 0 "#PWR034" H 6800 2300 50  0001 C CNN
+F 0 "#PWR036" H 6800 2300 50  0001 C CNN
 F 1 "GND" H 6800 2400 50  0000 C CNN
 F 2 "" H 6800 2550 50  0000 C CNN
@@
 Connection ~ 6200 2500
 $Comp
-L +3.3V #PWR035
+L +3.3V #PWR037
 U 1 1 589F6792
 P 6200 2100
-F 0 "#PWR035" H 6200 1950 50  0001 C CNN
+F 0 "#PWR037" H 6200 1950 50  0001 C CNN
 F 1 "+3.3V" H 6200 2240 50  0000 C CNN
 F 2 "" H 6200 2100 50  0000 C CNN
@@
 F 0 "C13" H 4810 3070 50  0000 L CNN
 F 1 "0.1uF" H 4810 2920 50  0000 L CNN
-F 2 "" H 4800 3000 50  0000 C CNN
+F 2 "robocon_pcb:SM0805_EXP0.5mm" H 4800 3000 50  0001 C CNN
 F 3 "" H 4800 3000 50  0000 C CNN
 	1    4800 3000
@@
 	4700 3000 4500 3000
 $Comp
-L GND #PWR036
+L GND #PWR038
 U 1 1 589F6831
 P 4500 3000
-F 0 "#PWR036" H 4500 2750 50  0001 C CNN
+F 0 "#PWR038" H 4500 2750 50  0001 C CNN
 F 1 "GND" H 4500 2850 50  0000 C CNN
 F 2 "" H 4500 3000 50  0000 C CNN
@@
 F 0 "J4" H 3600 3150 50  0000 C CNN
 F 1 "RJ12" H 3250 3150 50  0000 C CNN
-F 2 "" H 3400 2650 50  0000 C CNN
+F 2 "robocon_pcb:MODULAR-JACK_6P6C" H 3400 2650 50  0001 C CNN
 F 3 "" H 3400 2650 50  0000 C CNN
 	1    3400 2650
@@
 F 0 "J3" H 2650 3150 50  0000 C CNN
 F 1 "RJ12" H 2300 3150 50  0000 C CNN
-F 2 "" H 2450 2650 50  0000 C CNN
+F 2 "robocon_pcb:MODULAR-JACK_6P6C" H 2450 2650 50  0001 C CNN
 F 3 "" H 2450 2650 50  0000 C CNN
 	1    2450 2650
@@
 	2450 3100 2450 3150
 $Comp
-L GND #PWR037
+L GND #PWR039
 U 1 1 589F6C63
 P 2450 3150
-F 0 "#PWR037" H 2450 2900 50  0001 C CNN
+F 0 "#PWR039" H 2450 2900 50  0001 C CNN
 F 1 "GND" H 2450 3000 50  0000 C CNN
 F 2 "" H 2450 3150 50  0000 C CNN
@@
 $EndComp
 $Comp
-L GND #PWR038
+L GND #PWR040
 U 1 1 589F6C8D
 P 3400 3150
-F 0 "#PWR038" H 3400 2900 50  0001 C CNN
+F 0 "#PWR040" H 3400 2900 50  0001 C CNN
 F 1 "GND" H 3400 3000 50  0000 C CNN
 F 2 "" H 3400 3150 50  0000 C CNN
@@
 	2950 3200 2950 2900
 $Comp
-L +5V #PWR039
+L +5V #PWR041
 U 1 1 589F6D4F
 P 2950 2900
-F 0 "#PWR039" H 2950 2750 50  0001 C CNN
+F 0 "#PWR041" H 2950 2750 50  0001 C CNN
 F 1 "+5V" H 2950 3040 50  0000 C CNN
 F 2 "" H 2950 2900 50  0000 C CNN
@@
 $EndComp
 $Comp
-L +5V #PWR040
+L +5V #PWR042
 U 1 1 589F6D79
 P 2000 2900
-F 0 "#PWR040" H 2000 2750 50  0001 C CNN
+F 0 "#PWR042" H 2000 2750 50  0001 C CNN
 F 1 "+5V" H 2000 3040 50  0000 C CNN
 F 2 "" H 2000 2900 50  0000 C CNN
