File: STM32F4-MotherBoard_5.0.0/STM32F4-MotherBoard_5.0.0.sch (KiCad schematic (older format))
At the start: 2 parts

Commit message: LED
Changed lines of the file:
@@
 $Descr A3 16535 11693
 encoding utf-8
-Sheet 1 9
+Sheet 1 10
 Title ""
 Date ""
@@
 F1 "OSC.sch" 79
 $EndSheet
+$Sheet
+S 15050 5700 500  150
+U 589F8488
+F0 "LED" 79
+F1 "LED.sch" 79
+$EndSheet
 $EndSCHEMATC

Commit message: add run write
Connections:
- net NRST: now reaches U?.14 (NRST)
- net Write: now reaches U?.94 (BOOT0)
Changed lines of the file:
@@
 F1 "LED.sch" 79
 $EndSheet
+Wire Wire Line
+	2650 3350 2350 3350
+Text GLabel 2350 3350 0    60   Input ~ 0
+Write
+Wire Wire Line
+	2650 3550 2350 3550
+Text GLabel 2350 3550 0    60   Input ~ 0
+NRST
 $EndSCHEMATC
