File: STM32F4-MotherBoard_5.0.0/STM32F4-MotherBoard_5.0.0.sch (KiCad schematic (older format))
At the start: 2 parts

Commit message: 大枠の電源
Parts:
- added C? (x2): 2.2uF, symbol C
- added C? (x3): 0.1uF, symbol C
Connections:
- net power is gone; now on net +3V3: U?.100 (VDD), U?.11 (VDD), U?.19 (VDD), U?.28 (VDD), U?.50 (VDD), U?.75 (VDD)
- net GND: now also U?.10 (VSS), U?.20 (VSSA), U?.27 (VSS), U?.74 (VSS), U?.99 (VSS), C?.2, C?.2, C?.2, C?.2, C?.2
- net +3V3: now reaches U?.21 (VREF+)
- net +3V3: now also U?.22 (VDDA), U?.6 (VBAT), C?.1, C?.1, C?.1
- net at U?.49 (VCAP_1): now also C?.1
- net at U?.73 (VCAP_2): now also C?.1
Changed lines of the file:
@@
 	8050 2850 8050 2800
 Connection ~ 8050 2800
-Wire Wire Line
-	6850 2550 7000 2550
 Connection ~ 6850 2800
-Text GLabel 7000 2550 2    60   Input ~ 0
-power
 Text GLabel 2350 5150 0    60   Input ~ 0
 ENC0_Z
@@
 Text GLabel 2350 3550 0    60   Output ~ 0
 NRST
+Wire Wire Line
+	7250 8850 7250 8950
+Wire Wire Line
+	7250 8950 8050 8950
+Wire Wire Line
+	8050 8950 8050 8850
+Wire Wire Line
+	7850 8850 7850 8950
+Connection ~ 7850 8950
+Wire Wire Line
+	7650 8850 7650 9150
+Connection ~ 7650 8950
+Wire Wire Line
+	7450 8850 7450 8950
+Connection ~ 7450 8950
+$Comp
+L C C?
+U 1 1 589FAA7C
+P 8550 9050
+F 0 "C?" H 8575 9150 50  0000 L CNN
+F 1 "2.2uF" H 8575 8950 50  0000 L CNN
+F 2 "" H 8588 8900 50  0000 C CNN
+F 3 "" H 8550 9050 50  0000 C CNN
+	1    8550 9050
+	1    0    0    -1
+$EndComp
+$Comp
+L C C?
+U 1 1 589FAAA6
+P 9050 9050
+F 0 "C?" H 9075 9150 50  0000 L CNN
+F 1 "2.2uF" H 9075 8950 50  0000 L CNN
+F 2 "" H 9088 8900 50  0000 C CNN
+F 3 "" H 9050 9050 50  0000 C CNN
+	1    9050 9050
+	1    0    0    -1
+$EndComp
+Wire Wire Line
+	9050 8850 9050 8900
+Wire Wire Line
+	8550 8850 8550 8900
+Wire Wire Line
+	8550 9200 8550 9250
+Wire Wire Line
+	8550 9250 9050 9250
+Wire Wire Line
+	9050 9250 9050 9200
+Wire Wire Line
+	8800 9250 8800 9350
+Connection ~ 8800 9250
+$Comp
+L GND #PWR?
+U 1 1 589FACC4
+P 8800 9350
+F 0 "#PWR?" H 8800 9100 50  0001 C CNN
+F 1 "GND" H 8800 9200 50  0000 C CNN
+F 2 "" H 8800 9350 50  0000 C CNN
+F 3 "" H 8800 9350 50  0000 C CNN
+	1    8800 9350
+	1    0    0    -1
+$EndComp
+$Comp
+L GND #PWR?
+U 1 1 589FACE2
+P 7650 9150
+F 0 "#PWR?" H 7650 8900 50  0001 C CNN
+F 1 "GND" H 7650 9000 50  0000 C CNN
+F 2 "" H 7650 9150 50  0000 C CNN
+F 3 "" H 7650 9150 50  0000 C CNN
+	1    7650 9150
+	1    0    0    -1
+$EndComp
+$Comp
+L +3.3V #PWR?
+U 1 1 589FAD4B
+P 5350 2150
+F 0 "#PWR?" H 5350 2000 50  0001 C CNN
+F 1 "+3.3V" H 5350 2290 50  0000 C CNN
+F 2 "" H 5350 2150 50  0000 C CNN
+F 3 "" H 5350 2150 50  0000 C CNN
+	1    5350 2150
+	1    0    0    -1
+$EndComp
+$Comp
+L +3.3V #PWR?
+U 1 1 589FAD69
+P 5850 2150
+F 0 "#PWR?" H 5850 2000 50  0001 C CNN
+F 1 "+3.3V" H 5850 2290 50  0000 C CNN
+F 2 "" H 5850 2150 50  0000 C CNN
+F 3 "" H 5850 2150 50  0000 C CNN
+	1    5850 2150
+	1    0    0    -1
+$EndComp
+Wire Wire Line
+	5850 2150 5850 2850
+Wire Wire Line
+	5350 2150 5350 2850
+Wire Wire Line
+	5350 2350 5050 2350
+Wire Wire Line
+	5050 2350 5050 2450
+Connection ~ 5350 2350
+$Comp
+L C C?
+U 1 1 589FAEE5
+P 5050 2600
+F 0 "C?" H 5075 2700 50  0000 L CNN
+F 1 "0.1uF" H 5075 2500 50  0000 L CNN
+F 2 "" H 5088 2450 50  0000 C CNN
+F 3 "" H 5050 2600 50  0000 C CNN
+	1    5050 2600
+	1    0    0    -1
+$EndComp
+Wire Wire Line
+	5850 2350 5600 2350
+Wire Wire Line
+	5600 2350 5600 2450
+Connection ~ 5850 2350
+$Comp
+L C C?
+U 1 1 589FAF86
+P 5600 2600
+F 0 "C?" H 5625 2700 50  0000 L CNN
+F 1 "0.1uF" H 5625 2500 50  0000 L CNN
+F 2 "" H 5638 2450 50  0000 C CNN
+F 3 "" H 5600 2600 50  0000 C CNN
+	1    5600 2600
+	1    0    0    -1
+$EndComp
+Wire Wire Line
+	5050 2750 5050 2800
+Wire Wire Line
+	5600 2750 5600 2800
+$Comp
+L GND #PWR?
+U 1 1 589FB0D0
+P 5600 2800
+F 0 "#PWR?" H 5600 2550 50  0001 C CNN
+F 1 "GND" H 5600 2650 50  0000 C CNN
+F 2 "" H 5600 2800 50  0000 C CNN
+F 3 "" H 5600 2800 50  0000 C CNN
+	1    5600 2800
+	1    0    0    -1
+$EndComp
+$Comp
+L GND #PWR?
+U 1 1 589FB0F4
+P 5050 2800
+F 0 "#PWR?" H 5050 2550 50  0001 C CNN
+F 1 "GND" H 5050 2650 50  0000 C CNN
+F 2 "" H 5050 2800 50  0000 C CNN
+F 3 "" H 5050 2800 50  0000 C CNN
+	1    5050 2800
+	1    0    0    -1
+$EndComp
+$Comp
+L +3.3V #PWR?
+U 1 1 589FB171
+P 6850 2550
+F 0 "#PWR?" H 6850 2400 50  0001 C CNN
+F 1 "+3.3V" H 6850 2690 50  0000 C CNN
+F 2 "" H 6850 2550 50  0000 C CNN
+F 3 "" H 6850 2550 50  0000 C CNN
+	1    6850 2550
+	1    0    0    -1
+$EndComp
+$Comp
+L +3.3V #PWR?
+U 1 1 589FB1D7
+P 8850 2150
+F 0 "#PWR?" H 8850 2000 50  0001 C CNN
+F 1 "+3.3V" H 8850 2290 50  0000 C CNN
+F 2 "" H 8850 2150 50  0000 C CNN
+F 3 "" H 8850 2150 50  0000 C CNN
+	1    8850 2150
+	1    0    0    -1
+$EndComp
+Wire Wire Line
+	8850 2150 8850 2850
+Wire Wire Line
+	8850 2350 8600 2350
+Wire Wire Line
+	8600 2350 8600 2450
+Connection ~ 8850 2350
+$Comp
+L C C?
+U 1 1 589FB1E1
+P 8600 2600
+F 0 "C?" H 8625 2700 50  0000 L CNN
+F 1 "0.1uF" H 8625 2500 50  0000 L CNN
+F 2 "" H 8638 2450 50  0000 C CNN
+F 3 "" H 8600 2600 50  0000 C CNN
+	1    8600 2600
+	1    0    0    -1
+$EndComp
+$Comp
+L GND #PWR?
+U 1 1 589FB1F9
+P 8600 2800
+F 0 "#PWR?" H 8600 2550 50  0001 C CNN
+F 1 "GND" H 8600 2650 50  0000 C CNN
+F 2 "" H 8600 2800 50  0000 C CNN
+F 3 "" H 8600 2800 50  0000 C CNN
+	1    8600 2800
+	1    0    0    -1
+$EndComp
+Wire Wire Line
+	8600 2800 8600 2750
 $EndSCHEMATC

Commit message: SDとCANの追加とラベルミス修正
Connections:
- net SPI_SCK: now reaches U?.52 (PB13/SPI2_SCK/I2S2_CK/USART3_CTS/TIM1_CH1N/CAN2_TX/OTG_HS_ULPI_D6/ETH_RMII_TXD1/ETH_MII_TXD1/EVENTOUT)
- net SPI_MISO: now reaches U?.53 (PB14/SPI2_MISO/TIM1_CH2N/TIM12_CH1/OTG_HS_DM/USART3_RTS/TIM8_CH2N/I2S2ext_SD/EVENTOUT)
- net SPI_MOSI: now reaches U?.54 (PB15/SPI2_MOSI/I2S2_SD/TIM1_CH3N/TIM8_CH3N/TIM12_CH2/OTG_HS_DP/EVENTOUT)
Changed lines of the file:
@@
 $Descr A3 16535 11693
 encoding utf-8
-Sheet 1 10
+Sheet 1 11
 Title ""
 Date ""
@@
 Wire Wire Line
 	8600 2800 8600 2750
+Text GLabel 2350 8250 0    60   Output ~ 0
+SPI_SCK
+Text GLabel 2350 8350 0    60   Input ~ 0
+SPI_MISO
+Text GLabel 2350 8450 0    60   Output ~ 0
+SPI_MOSI
+$Sheet
+S 15100 6150 500  150
+U 58A2FD89
+F0 "SD" 79
+F1 "SD.sch" 79
+$EndSheet
 $EndSCHEMATC

Commit message: 回路図終わり
Parts:
- gave numbers to parts that had none: 7
Connections:
- net SPI_CS: now reaches U1.7 (PC13/EVENTOUT)
- net pushSW renamed PushSW
- no-connect marks 3 -> 2
Changed lines of the file:
@@
 $Descr A3 16535 11693
 encoding utf-8
-Sheet 1 11
+Sheet 1 12
 Title ""
 Date ""
@@
 $EndSheet
 $Comp
-L STM32F407VG U?
+L STM32F407VG U1
 U 1 1 589AAFA6
 P 7650 5850
-F 0 "U?" H 7650 5850 50  0000 C CNN
+F 0 "U1" H 7650 5850 50  0000 C CNN
 F 1 "STM32F407VG" H 7650 5950 50  0000 C CNN
 F 2 "TQFP100" H 7650 5750 50  0000 C CNN
@@
 CAN_TX
 Text GLabel 2350 7950 0    60   Input ~ 0
-pushSW
+PushSW
 Text GLabel 2350 8050 0    60   BiDi ~ 0
 DIO0_2
@@
 Text GLabel 12950 8050 2    60   BiDi ~ 0
 DIO1_2
-NoConn ~ 12650 8250
 NoConn ~ 12650 8350
 NoConn ~ 12650 8450
@@
 	1600 7150 1600 7350
 $Comp
-L R R?
+L R R1
 U 1 1 589F1F0A
 P 1600 7500
-F 0 "R?" V 1680 7500 50  0000 C CNN
+F 0 "R1" V 1680 7500 50  0000 C CNN
 F 1 "100k" V 1600 7500 50  0000 C CNN
 F 2 "" V 1530 7500 50  0000 C CNN
@@
 	1600 7650 1600 7750
 $Comp
-L GND #PWR?
+L GND #PWR01
 U 1 1 589F1F9C
 P 1600 7750
-F 0 "#PWR?" H 1600 7500 50  0001 C CNN
+F 0 "#PWR01" H 1600 7500 50  0001 C CNN
 F 1 "GND" H 1600 7600 50  0000 C CNN
 F 2 "" H 1600 7750 50  0000 C CNN
@@
 Connection ~ 7450 8950
 $Comp
-L C C?
+L C C3
 U 1 1 589FAA7C
 P 8550 9050
-F 0 "C?" H 8575 9150 50  0000 L CNN
+F 0 "C3" H 8575 9150 50  0000 L CNN
 F 1 "2.2uF" H 8575 8950 50  0000 L CNN
 F 2 "" H 8588 8900 50  0000 C CNN
@@
 $EndComp
 $Comp
-L C C?
+L C C5
 U 1 1 589FAAA6
 P 9050 9050
-F 0 "C?" H 9075 9150 50  0000 L CNN
+F 0 "C5" H 9075 9150 50  0000 L CNN
 F 1 "2.2uF" H 9075 8950 50  0000 L CNN
 F 2 "" H 9088 8900 50  0000 C CNN
@@
 Connection ~ 8800 9250
 $Comp
-L GND #PWR?
+L GND #PWR02
 U 1 1 589FACC4
 P 8800 9350
-F 0 "#PWR?" H 8800 9100 50  0001 C CNN
+F 0 "#PWR02" H 8800 9100 50  0001 C CNN
 F 1 "GND" H 8800 9200 50  0000 C CNN
 F 2 "" H 8800 9350 50  0000 C CNN
@@
 $EndComp
 $Comp
-L GND #PWR?
+L GND #PWR03
 U 1 1 589FACE2
 P 7650 9150
-F 0 "#PWR?" H 7650 8900 50  0001 C CNN
+F 0 "#PWR03" H 7650 8900 50  0001 C CNN
 F 1 "GND" H 7650 9000 50  0000 C CNN
 F 2 "" H 7650 9150 50  0000 C CNN
@@
 $EndComp
 $Comp
-L +3.3V #PWR?
+L +3.3V #PWR04
 U 1 1 589FAD4B
 P 5350 2150
-F 0 "#PWR?" H 5350 2000 50  0001 C CNN
+F 0 "#PWR04" H 5350 2000 50  0001 C CNN
 F 1 "+3.3V" H 5350 2290 50  0000 C CNN
 F 2 "" H 5350 2150 50  0000 C CNN
@@
 $EndComp
 $Comp
-L +3.3V #PWR?
+L +3.3V #PWR05
 U 1 1 589FAD69
 P 5850 2150
-F 0 "#PWR?" H 5850 2000 50  0001 C CNN
+F 0 "#PWR05" H 5850 2000 50  0001 C CNN
 F 1 "+3.3V" H 5850 2290 50  0000 C CNN
 F 2 "" H 5850 2150 50  0000 C CNN
@@
 Connection ~ 5350 2350
 $Comp
-L C C?
+L C C1
 U 1 1 589FAEE5
 P 5050 2600
-F 0 "C?" H 5075 2700 50  0000 L CNN
+F 0 "C1" H 5075 2700 50  0000 L CNN
 F 1 "0.1uF" H 5075 2500 50  0000 L CNN
 F 2 "" H 5088 2450 50  0000 C CNN
@@
 Connection ~ 5850 2350
 $Comp
-L C C?
+L C C2
 U 1 1 589FAF86
 P 5600 2600
-F 0 "C?" H 5625 2700 50  0000 L CNN
+F 0 "C2" H 5625 2700 50  0000 L CNN
 F 1 "0.1uF" H 5625 2500 50  0000 L CNN
 F 2 "" H 5638 2450 50  0000 C CNN
@@
 	5600 2750 5600 2800
 $Comp
-L GND #PWR?
+L GND #PWR06
 U 1 1 589FB0D0
 P 5600 2800
-F 0 "#PWR?" H 5600 2550 50  0001 C CNN
+F 0 "#PWR06" H 5600 2550 50  0001 C CNN
 F 1 "GND" H 5600 2650 50  0000 C CNN
 F 2 "" H 5600 2800 50  0000 C CNN
@@
 $EndComp
 $Comp
-L GND #PWR?
+L GND #PWR07
 U 1 1 589FB0F4
 P 5050 2800
-F 0 "#PWR?" H 5050 2550 50  0001 C CNN
+F 0 "#PWR07" H 5050 2550 50  0001 C CNN
 F 1 "GND" H 5050 2650 50  0000 C CNN
 F 2 "" H 5050 2800 50  0000 C CNN
@@
 $EndComp
 $Comp
-L +3.3V #PWR?
+L +3.3V #PWR08
 U 1 1 589FB171
 P 6850 2550
-F 0 "#PWR?" H 6850 2400 50  0001 C CNN
+F 0 "#PWR08" H 6850 2400 50  0001 C CNN
 F 1 "+3.3V" H 6850 2690 50  0000 C CNN
 F 2 "" H 6850 2550 50  0000 C CNN
@@
 $EndComp
 $Comp
-L +3.3V #PWR?
+L +3.3V #PWR09
 U 1 1 589FB1D7
 P 8850 2150
-F 0 "#PWR?" H 8850 2000 50  0001 C CNN
+F 0 "#PWR09" H 8850 2000 50  0001 C CNN
 F 1 "+3.3V" H 8850 2290 50  0000 C CNN
 F 2 "" H 8850 2150 50  0000 C CNN
@@
 Connection ~ 8850 2350
 $Comp
-L C C?
+L C C4
 U 1 1 589FB1E1
 P 8600 2600
-F 0 "C?" H 8625 2700 50  0000 L CNN
+F 0 "C4" H 8625 2700 50  0000 L CNN
 F 1 "0.1uF" H 8625 2500 50  0000 L CNN
 F 2 "" H 8638 2450 50  0000 C CNN
@@
 $EndComp
 $Comp
-L GND #PWR?
+L GND #PWR010
 U 1 1 589FB1F9
 P 8600 2800
-F 0 "#PWR?" H 8600 2550 50  0001 C CNN
+F 0 "#PWR010" H 8600 2550 50  0001 C CNN
 F 1 "GND" H 8600 2650 50  0000 C CNN
 F 2 "" H 8600 2800 50  0000 C CNN
@@
 F1 "SD.sch" 79
 $EndSheet
+Wire Wire Line
+	12650 8250 12950 8250
+Text GLabel 12950 8250 2    60   Output ~ 0
+SPI_CS
+$Sheet
+S 15150 6600 500  150
+U 58A5790E
+F0 "ENC" 79
+F1 "ENC.sch" 79
+$EndSheet
 $EndSCHEMATC

Commit message: 部品名変更
Parts:
- C1, C2, C3, C4, C5: footprint (none) -> robocon_pcb:SM0805_EXP0.5mm
- R1: footprint (none) -> robocon_pcb:SM0603_EXP0.5mm
- U1: symbol STM32F407VG -> STM32F407VG-RESCUE-STM32F4-MotherBoard_5.0.0
Changed lines of the file:
@@
 EESchema Schematic File Version 2
+LIBS:STM32F4-MotherBoard_5.0.0-rescue
 LIBS:power
 LIBS:device
@@
 $EndSheet
 $Comp
-L STM32F407VG U1
+L STM32F407VG-RESCUE-STM32F4-MotherBoard_5.0.0 U1
 U 1 1 589AAFA6
 P 7650 5850
@@
 F 0 "R1" V 1680 7500 50  0000 C CNN
 F 1 "100k" V 1600 7500 50  0000 C CNN
-F 2 "" V 1530 7500 50  0000 C CNN
+F 2 "robocon_pcb:SM0603_EXP0.5mm" V 1530 7500 50  0001 C CNN
 F 3 "" H 1600 7500 50  0000 C CNN
 	1    1600 7500
@@
 F 0 "C3" H 8575 9150 50  0000 L CNN
 F 1 "2.2uF" H 8575 8950 50  0000 L CNN
-F 2 "" H 8588 8900 50  0000 C CNN
+F 2 "robocon_pcb:SM0805_EXP0.5mm" H 8588 8900 50  0001 C CNN
 F 3 "" H 8550 9050 50  0000 C CNN
 	1    8550 9050
@@
 F 0 "C5" H 9075 9150 50  0000 L CNN
 F 1 "2.2uF" H 9075 8950 50  0000 L CNN
-F 2 "" H 9088 8900 50  0000 C CNN
+F 2 "robocon_pcb:SM0805_EXP0.5mm" H 9088 8900 50  0001 C CNN
 F 3 "" H 9050 9050 50  0000 C CNN
 	1    9050 9050
@@
 F 0 "C1" H 5075 2700 50  0000 L CNN
 F 1 "0.1uF" H 5075 2500 50  0000 L CNN
-F 2 "" H 5088 2450 50  0000 C CNN
+F 2 "robocon_pcb:SM0805_EXP0.5mm" H 5088 2450 50  0001 C CNN
 F 3 "" H 5050 2600 50  0000 C CNN
 	1    5050 2600
@@
 F 0 "C2" H 5625 2700 50  0000 L CNN
 F 1 "0.1uF" H 5625 2500 50  0000 L CNN
-F 2 "" H 5638 2450 50  0000 C CNN
+F 2 "robocon_pcb:SM0805_EXP0.5mm" H 5638 2450 50  0001 C CNN
 F 3 "" H 5600 2600 50  0000 C CNN
 	1    5600 2600
@@
 F 0 "C4" H 8625 2700 50  0000 L CNN
 F 1 "0.1uF" H 8625 2500 50  0000 L CNN
-F 2 "" H 8638 2450 50  0000 C CNN
+F 2 "robocon_pcb:SM0805_EXP0.5mm" H 8638 2450 50  0001 C CNN
 F 3 "" H 8600 2600 50  0000 C CNN
 	1    8600 2600

Commit message: 関連付けできたの
Parts:
- U1: footprint TQFP100 -> Housings_QFP:LQFP-100_14x14mm_Pitch0.5mm
Changed lines of the file:
@@
 F 0 "U1" H 7650 5850 50  0000 C CNN
 F 1 "STM32F407VG" H 7650 5950 50  0000 C CNN
-F 2 "TQFP100" H 7650 5750 50  0000 C CNN
+F 2 "Housings_QFP:LQFP-100_14x14mm_Pitch0.5mm" H 7650 5750 50  0000 C CNN
 F 3 "" H 7650 5850 50  0000 C CNN
 	1    7650 5850
