File: STM32F4-MotherBoard_5.0.0/ENC.sch (KiCad schematic (older format))
At the start: 12 parts, among them P7 ENC0, P8 ENC2, P9 ENC1

Commit message: ミス
Changed lines of the file:
@@
 L +12V #PWR075
 U 1 1 58A57A8C
-P 3500 2600
-F 0 "#PWR075" H 3500 2450 50  0001 C CNN
-F 1 "+12V" H 3500 2740 50  0000 C CNN
-F 2 "" H 3500 2600 50  0000 C CNN
-F 3 "" H 3500 2600 50  0000 C CNN
-	1    3500 2600
-	1    0    0    -1
-$EndComp
-Wire Wire Line
-	3500 2600 3500 2950
+P 3500 2550
+F 0 "#PWR075" H 3500 2400 50  0001 C CNN
+F 1 "+12V" H 3500 2690 50  0000 C CNN
+F 2 "" H 3500 2550 50  0000 C CNN
+F 3 "" H 3500 2550 50  0000 C CNN
+	1    3500 2550
+	1    0    0    -1
+$EndComp
+Wire Wire Line
+	3500 2550 3500 2950
 Wire Wire Line
 	3500 2950 3550 2950
@@
 L +12V #PWR078
 U 1 1 58A57D7D
-P 4900 3450
-F 0 "#PWR078" H 4900 3300 50  0001 C CNN
-F 1 "+12V" H 4900 3590 50  0000 C CNN
-F 2 "" H 4900 3450 50  0000 C CNN
-F 3 "" H 4900 3450 50  0000 C CNN
-	1    4900 3450
-	1    0    0    -1
-$EndComp
-Wire Wire Line
-	4900 3450 4900 3800
+P 4900 3400
+F 0 "#PWR078" H 4900 3250 50  0001 C CNN
+F 1 "+12V" H 4900 3540 50  0000 C CNN
+F 2 "" H 4900 3400 50  0000 C CNN
+F 3 "" H 4900 3400 50  0000 C CNN
+	1    4900 3400
+	1    0    0    -1
+$EndComp
 Wire Wire Line
 	4900 3800 4950 3800
@@
 L +12V #PWR081
 U 1 1 58A57E7F
-P 3600 4750
-F 0 "#PWR081" H 3600 4600 50  0001 C CNN
-F 1 "+12V" H 3600 4890 50  0000 C CNN
-F 2 "" H 3600 4750 50  0000 C CNN
-F 3 "" H 3600 4750 50  0000 C CNN
-	1    3600 4750
-	1    0    0    -1
-$EndComp
-Wire Wire Line
-	3600 4750 3600 5100
+P 3600 4700
+F 0 "#PWR081" H 3600 4550 50  0001 C CNN
+F 1 "+12V" H 3600 4840 50  0000 C CNN
+F 2 "" H 3600 4700 50  0000 C CNN
+F 3 "" H 3600 4700 50  0000 C CNN
+	1    3600 4700
+	1    0    0    -1
+$EndComp
 Wire Wire Line
 	3600 5100 3650 5100
@@
 	1    0    0    -1
 $EndComp
+Wire Wire Line
+	4900 3400 4900 3800
+Wire Wire Line
+	3600 4700 3600 5100
 $EndSCHEMATC
