File: STM32F4-MotherBoard_5.0.0/LED.sch (KiCad schematic (older format))
At the start: 4 parts

Commit message: LED
Parts:
- removed C? (x2): 22uF, symbol C_Small
- removed R?: 220, symbol R
- removed Y?: 8MHz, symbol Crystal
- added D?: LED, symbol LED
- added R?: 1k, symbol R
Connections:
- net GND: now also R?.2
- new net: D?.1 (K), R?.1
- new net LED: D?.2 (A)
Changed lines of the file:
@@
 $Descr A4 11693 8268
 encoding utf-8
-Sheet 9 10
+Sheet 10 10
 Title ""
 Date ""
@@
 Comment4 ""
 $EndDescr
-Text GLabel 4100 2500 0    60   Input ~ 0
-OSC_IN
-Text GLabel 4100 3100 0    60   Input ~ 0
-OSC_OUT
+Text GLabel 3700 2500 0    60   Input ~ 0
+LED
 $Comp
-L Crystal Y?
-U 1 1 589F7562
-P 4600 2800
-F 0 "Y?" H 4600 2950 50  0000 C CNN
-F 1 "8MHz" H 4600 2650 50  0000 C CNN
-F 2 "" H 4600 2800 50  0000 C CNN
-F 3 "" H 4600 2800 50  0000 C CNN
-	1    4600 2800
-	0    1    1    0
+L LED D?
+U 1 1 589F8496
+P 4000 2500
+F 0 "D?" H 4000 2600 50  0000 C CNN
+F 1 "LED" H 4000 2400 50  0000 C CNN
+F 2 "" H 4000 2500 50  0000 C CNN
+F 3 "" H 4000 2500 50  0000 C CNN
+	1    4000 2500
+	-1   0    0    1
 $EndComp
 Wire Wire Line
-	4100 2500 4750 2500
+	3800 2500 3700 2500
 Wire Wire Line
-	4600 2500 4600 2650
+	4200 2500 4350 2500
 Wire Wire Line
-	4600 2950 4600 3100
+	4350 2500 4350 2550
 $Comp
 L R R?
-U 1 1 589F75A6
-P 4350 3100
-F 0 "R?" V 4430 3100 50  0000 C CNN
-F 1 "220" V 4350 3100 50  0000 C CNN
-F 2 "" V 4280 3100 50  0000 C CNN
-F 3 "" H 4350 3100 50  0000 C CNN
-	1    4350 3100
-	0    1    1    0
+U 1 1 589F84DD
+P 4350 2700
+F 0 "R?" V 4430 2700 50  0000 C CNN
+F 1 "1k" V 4350 2700 50  0000 C CNN
+F 2 "" V 4280 2700 50  0000 C CNN
+F 3 "" H 4350 2700 50  0000 C CNN
+	1    4350 2700
+	1    0    0    -1
 $EndComp
 Wire Wire Line
-	4200 3100 4100 3100
-Wire Wire Line
-	4500 3100 4750 3100
-$Comp
-L C_Small C?
-U 1 1 589F75D2
-P 4850 3100
-F 0 "C?" H 4860 3170 50  0000 L CNN
-F 1 "22uF" H 4860 3020 50  0000 L CNN
-F 2 "" H 4850 3100 50  0000 C CNN
-F 3 "" H 4850 3100 50  0000 C CNN
-	1    4850 3100
-	0    1    1    0
-$EndComp
-$Comp
-L C_Small C?
-U 1 1 589F75F6
-P 4850 2500
-F 0 "C?" H 4860 2570 50  0000 L CNN
-F 1 "22uF" H 4860 2420 50  0000 L CNN
-F 2 "" H 4850 2500 50  0000 C CNN
-F 3 "" H 4850 2500 50  0000 C CNN
-	1    4850 2500
-	0    1    1    0
-$EndComp
-Connection ~ 4600 2500
-Connection ~ 4600 3100
-Wire Wire Line
-	4950 3100 5050 3100
-Wire Wire Line
-	5050 2500 5050 3250
-Wire Wire Line
-	5050 2500 4950 2500
-Connection ~ 5050 3100
+	4350 2850 4350 2950
 $Comp
 L GND #PWR?
-U 1 1 589F765B
-P 5050 3250
-F 0 "#PWR?" H 5050 3000 50  0001 C CNN
-F 1 "GND" H 5050 3100 50  0000 C CNN
-F 2 "" H 5050 3250 50  0000 C CNN
-F 3 "" H 5050 3250 50  0000 C CNN
-	1    5050 3250
+U 1 1 589F8502
+P 4350 2950
+F 0 "#PWR?" H 4350 2700 50  0001 C CNN
+F 1 "GND" H 4350 2800 50  0000 C CNN
+F 2 "" H 4350 2950 50  0000 C CNN
+F 3 "" H 4350 2950 50  0000 C CNN
+	1    4350 2950
 	1    0    0    -1
 $EndComp

Commit message: 回路図終わり
Parts:
- gave numbers to parts that had none: 2
Changed lines of the file:
@@
 $Descr A4 11693 8268
 encoding utf-8
-Sheet 10 11
+Sheet 10 12
 Title ""
 Date ""
@@
 LED
 $Comp
-L LED D?
+L LED D2
 U 1 1 589F8496
 P 4000 2500
-F 0 "D?" H 4000 2600 50  0000 C CNN
+F 0 "D2" H 4000 2600 50  0000 C CNN
 F 1 "LED" H 4000 2400 50  0000 C CNN
 F 2 "" H 4000 2500 50  0000 C CNN
@@
 	4350 2500 4350 2550
 $Comp
-L R R?
+L R R39
 U 1 1 589F84DD
 P 4350 2700
-F 0 "R?" V 4430 2700 50  0000 C CNN
+F 0 "R39" V 4430 2700 50  0000 C CNN
 F 1 "1k" V 4350 2700 50  0000 C CNN
 F 2 "" V 4280 2700 50  0000 C CNN
@@
 	4350 2850 4350 2950
 $Comp
-L GND #PWR?
+L GND #PWR065
 U 1 1 589F8502
 P 4350 2950
-F 0 "#PWR?" H 4350 2700 50  0001 C CNN
+F 0 "#PWR065" H 4350 2700 50  0001 C CNN
 F 1 "GND" H 4350 2800 50  0000 C CNN
 F 2 "" H 4350 2950 50  0000 C CNN

Commit message: 部品名変更
Parts:
- D2: footprint (none) -> LEDs:LED_0603
- R39: footprint (none) -> robocon_pcb:SM0603_EXP0.5mm
Changed lines of the file:
@@
 EESchema Schematic File Version 2
+LIBS:STM32F4-MotherBoard_5.0.0-rescue
 LIBS:power
 LIBS:device
@@
 F 0 "D2" H 4000 2600 50  0000 C CNN
 F 1 "LED" H 4000 2400 50  0000 C CNN
-F 2 "" H 4000 2500 50  0000 C CNN
+F 2 "LEDs:LED_0603" H 4000 2500 50  0001 C CNN
 F 3 "" H 4000 2500 50  0000 C CNN
 	1    4000 2500
@@
 F 0 "R39" V 4430 2700 50  0000 C CNN
 F 1 "1k" V 4350 2700 50  0000 C CNN
-F 2 "" V 4280 2700 50  0000 C CNN
+F 2 "robocon_pcb:SM0603_EXP0.5mm" V 4280 2700 50  0001 C CNN
 F 3 "" H 4350 2700 50  0000 C CNN
 	1    4350 2700
@@
 	4350 2850 4350 2950
 $Comp
-L GND #PWR065
+L GND #PWR067
 U 1 1 589F8502
 P 4350 2950
-F 0 "#PWR065" H 4350 2700 50  0001 C CNN
+F 0 "#PWR067" H 4350 2700 50  0001 C CNN
 F 1 "GND" H 4350 2800 50  0000 C CNN
 F 2 "" H 4350 2950 50  0000 C CNN
