File: STM32F4-MotherBoard_5.0.0/OSC.sch (KiCad schematic (older format))
At the start: 4 parts

Commit message: 回路図終わり
Parts:
- gave numbers to parts that had none: 4
Changed lines of the file:
@@
 $Descr A4 11693 8268
 encoding utf-8
-Sheet 9 11
+Sheet 9 12
 Title ""
 Date ""
@@
 OSC_OUT
 $Comp
-L Crystal Y?
+L Crystal Y1
 U 1 1 589F7562
 P 4600 2800
-F 0 "Y?" H 4600 2950 50  0000 C CNN
+F 0 "Y1" H 4600 2950 50  0000 C CNN
 F 1 "8MHz" H 4600 2650 50  0000 C CNN
 F 2 "" H 4600 2800 50  0000 C CNN
@@
 	4600 2950 4600 3100
 $Comp
-L R R?
+L R R38
 U 1 1 589F75A6
 P 4350 3100
-F 0 "R?" V 4430 3100 50  0000 C CNN
+F 0 "R38" V 4430 3100 50  0000 C CNN
 F 1 "220" V 4350 3100 50  0000 C CNN
 F 2 "" V 4280 3100 50  0000 C CNN
@@
 	4500 3100 4750 3100
 $Comp
-L C_Small C?
+L C_Small C19
 U 1 1 589F75D2
 P 4850 3100
-F 0 "C?" H 4860 3170 50  0000 L CNN
+F 0 "C19" H 4860 3170 50  0000 L CNN
 F 1 "22uF" H 4860 3020 50  0000 L CNN
 F 2 "" H 4850 3100 50  0000 C CNN
@@
 $EndComp
 $Comp
-L C_Small C?
+L C_Small C18
 U 1 1 589F75F6
 P 4850 2500
-F 0 "C?" H 4860 2570 50  0000 L CNN
+F 0 "C18" H 4860 2570 50  0000 L CNN
 F 1 "22uF" H 4860 2420 50  0000 L CNN
 F 2 "" H 4850 2500 50  0000 C CNN
@@
 Connection ~ 5050 3100
 $Comp
-L GND #PWR?
+L GND #PWR064
 U 1 1 589F765B
 P 5050 3250
-F 0 "#PWR?" H 5050 3000 50  0001 C CNN
+F 0 "#PWR064" H 5050 3000 50  0001 C CNN
 F 1 "GND" H 5050 3100 50  0000 C CNN
 F 2 "" H 5050 3250 50  0000 C CNN

Commit message: 部品名変更
Parts:
- R38: footprint (none) -> robocon_pcb:SM0603_EXP0.5mm
Changed lines of the file:
@@
 EESchema Schematic File Version 2
+LIBS:STM32F4-MotherBoard_5.0.0-rescue
 LIBS:power
 LIBS:device
@@
 F 0 "Y1" H 4600 2950 50  0000 C CNN
 F 1 "8MHz" H 4600 2650 50  0000 C CNN
-F 2 "" H 4600 2800 50  0000 C CNN
+F 2 "" H 4600 2800 50  0001 C CNN
 F 3 "" H 4600 2800 50  0000 C CNN
 	1    4600 2800
@@
 F 0 "R38" V 4430 3100 50  0000 C CNN
 F 1 "220" V 4350 3100 50  0000 C CNN
-F 2 "" V 4280 3100 50  0000 C CNN
+F 2 "robocon_pcb:SM0603_EXP0.5mm" V 4280 3100 50  0001 C CNN
 F 3 "" H 4350 3100 50  0000 C CNN
 	1    4350 3100
@@
 F 0 "C19" H 4860 3170 50  0000 L CNN
 F 1 "22uF" H 4860 3020 50  0000 L CNN
-F 2 "" H 4850 3100 50  0000 C CNN
+F 2 "" H 4850 3100 50  0001 C CNN
 F 3 "" H 4850 3100 50  0000 C CNN
 	1    4850 3100
@@
 F 0 "C18" H 4860 2570 50  0000 L CNN
 F 1 "22uF" H 4860 2420 50  0000 L CNN
-F 2 "" H 4850 2500 50  0000 C CNN
+F 2 "" H 4850 2500 50  0001 C CNN
 F 3 "" H 4850 2500 50  0000 C CNN
 	1    4850 2500
@@
 Connection ~ 5050 3100
 $Comp
-L GND #PWR064
+L GND #PWR066
 U 1 1 589F765B
 P 5050 3250
-F 0 "#PWR064" H 5050 3000 50  0001 C CNN
+F 0 "#PWR066" H 5050 3000 50  0001 C CNN
 F 1 "GND" H 5050 3100 50  0000 C CNN
 F 2 "" H 5050 3250 50  0000 C CNN

Commit message: 関連付けできたの
Parts:
- C18, C19: footprint (none) -> robocon_pcb:SM0805_EXP0.5mm
- Y1: footprint (none) -> Crystals:Crystal_HC49-U_Vertical
Changed lines of the file:
@@
 F 0 "Y1" H 4600 2950 50  0000 C CNN
 F 1 "8MHz" H 4600 2650 50  0000 C CNN
-F 2 "" H 4600 2800 50  0001 C CNN
+F 2 "Crystals:Crystal_HC49-U_Vertical" H 4600 2800 50  0001 C CNN
 F 3 "" H 4600 2800 50  0000 C CNN
 	1    4600 2800
@@
 F 0 "C19" H 4860 3170 50  0000 L CNN
 F 1 "22uF" H 4860 3020 50  0000 L CNN
-F 2 "" H 4850 3100 50  0001 C CNN
+F 2 "robocon_pcb:SM0805_EXP0.5mm" H 4850 3100 50  0001 C CNN
 F 3 "" H 4850 3100 50  0000 C CNN
 	1    4850 3100
@@
 F 0 "C18" H 4860 2570 50  0000 L CNN
 F 1 "22uF" H 4860 2420 50  0000 L CNN
-F 2 "" H 4850 2500 50  0001 C CNN
+F 2 "robocon_pcb:SM0805_EXP0.5mm" H 4850 2500 50  0001 C CNN
 F 3 "" H 4850 2500 50  0000 C CNN
 	1    4850 2500
@@
 Connection ~ 5050 3100
 $Comp
-L GND #PWR066
+L GND #PWR070
 U 1 1 589F765B
 P 5050 3250
-F 0 "#PWR066" H 5050 3000 50  0001 C CNN
+F 0 "#PWR070" H 5050 3000 50  0001 C CNN
 F 1 "GND" H 5050 3100 50  0000 C CNN
 F 2 "" H 5050 3250 50  0000 C CNN
